File: NozzleControlBoard.kicad_pcb (KiCad board)
At the start: 4 copper layers, 345 x 346 mm, 364 parts, among them IC2 MAX3094EESE+, IC3 MAX22245BAWA+, J1 24V_OUT, J103 SHIFT_DATA_TOSS, J2 SHIFT_DATA_TOSS, J3 Conn_01x12_Male, J8 SOL1, Q1 TPN22006NH,LQ, U1 74HCT595, U10 AP2127K-3.3, U102 74HCT595, U103 TLP291, U104 TLP291, U105 TLP291, U106 TLP291, U107 TLP291, U108 TLP291, U109 TLP291, U11 ATmega8A-A, U110 TLP291, U12 TLP291, U13 TLP291, U14 TLP291, U15 TLP291, U16 TLP291, U17 TLP291, U18 TLP291, U2 74HCT595, U27 TLP291, U28 TLP291, U29 TLP291, U3 TLP291, U30 TLP291, U31 TLP291, U32 TLP291, U33 TLP291, U34 TLP291, U43 TLP291, U44 TLP291, U45 TLP291, U46 TLP291, U47 74HCT595, U56 TLP291, U57 TLP291, U58 TLP291, U59 TLP291, U6 TLP291, U60 TLP291, U61 TLP291, U62 TLP291, U63 TLP291, U64 74HCT595, U7 TLP291, U73 TLP291, U74 TLP291, U75 TLP291, U76 TLP291, U77 TLP291, U78 TLP291, U79 TLP291, U8 TLP291, U80 TLP291, U81 74HCT595, U87 SOL14, U9 TLP291, Y1 Crystal_GND24

Commit message: .
.
Parts:
- added J10: SOL3, footprint:2PIN, B.Cu at (305.8, -417.1)
- added J11: SOL4, footprint:2PIN, B.Cu at (304.6, -328.0)
- added J12: SOL5, footprint:2PIN, B.Cu at (295.5, -417.3)
- added J13: SOL6, footprint:2PIN, B.Cu at (293.9, -327.9)
- added J14: SOL7, footprint:2PIN, B.Cu at (284.8, -417.3)
- added J15: SOL8, footprint:2PIN, B.Cu at (283.2, -327.9)
- added J16: SOL9, footprint:2PIN, B.Cu at (265.7, -417.1)
- added J17: SOL10, footprint:2PIN, B.Cu at (264.3, -327.9)
- added J18: SOL11, footprint:2PIN, B.Cu at (254.0, -417.1)
- added J19: SOL12, footprint:2PIN, B.Cu at (253.2, -327.9)
- added J20: SOL13, footprint:2PIN, B.Cu at (242.3, -417.0)
- added J21: SOL14, footprint:2PIN, B.Cu at (242.2, -327.9)
- added J22: SOL15, footprint:2PIN, B.Cu at (230.5, -417.2)
- added J23: SOL16, footprint:2PIN, B.Cu at (231.2, -327.9)
- added J24: SOL17, footprint:2PIN, B.Cu at (216.7, -417.1)
- added J25: SOL18, footprint:2PIN, B.Cu at (217.0, -328.1)
- added J26: SOL19, footprint:2PIN, B.Cu at (203.8, -417.1)
- added J27: SOL20, footprint:2PIN, B.Cu at (203.7, -327.8)
- added J28: SOL21, footprint:2PIN, B.Cu at (190.7, -417.1)
- added J29: SOL22, footprint:2PIN, B.Cu at (187.5, -327.2)
- added J30: SOL23, footprint:2PIN, B.Cu at (177.8, -417.2)
- added J31: SOL24, footprint:2PIN, F.Cu at (170.0, -327.4)
- added J9: SOL2, footprint:2PIN, B.Cu at (315.3, -327.7)
- added Q10: TPN22006NH,LQ, footprint:TPN22006NHLQ, F.Cu at (261.9, -338.9)
- added Q11: TPN22006NH,LQ, footprint:TPN22006NHLQ, F.Cu at (256.4, -406.3)
- added Q12: TPN22006NH,LQ, footprint:TPN22006NHLQ, F.Cu at (250.7, -338.8)
- added Q13: TPN22006NH,LQ, footprint:TPN22006NHLQ, F.Cu at (244.6, -406.1)
- added Q14: TPN22006NH,LQ, footprint:TPN22006NHLQ, F.Cu at (239.8, -338.9)
- added Q15: TPN22006NH,LQ, footprint:TPN22006NHLQ, F.Cu at (232.8, -406.3)
- added Q16: TPN22006NH,LQ, footprint:TPN22006NHLQ, F.Cu at (228.7, -338.8)
- added Q17: TPN22006NH,LQ, footprint:TPN22006NHLQ, F.Cu at (219.1, -406.2)
- added Q18: TPN22006NH,LQ, footprint:TPN22006NHLQ, F.Cu at (214.6, -338.9)
- added Q19: TPN22006NH,LQ, footprint:TPN22006NHLQ, F.Cu at (206.1, -406.3)
- added Q2: TPN22006NH,LQ, footprint:TPN22006NHLQ, F.Cu at (312.9, -338.6)
- added Q20: TPN22006NH,LQ, footprint:TPN22006NHLQ, F.Cu at (201.3, -338.7)
- added Q21: TPN22006NH,LQ, footprint:TPN22006NHLQ, F.Cu at (193.1, -406.2)
- added Q22: TPN22006NH,LQ, footprint:TPN22006NHLQ, F.Cu at (185.1, -338.2)
- added Q23: TPN22006NH,LQ, footprint:TPN22006NHLQ, F.Cu at (180.2, -406.2)
- added Q24: TPN22006NH,LQ, footprint:TPN22006NHLQ, F.Cu at (170.3, -338.4)
- added Q3: TPN22006NH,LQ, footprint:TPN22006NHLQ, F.Cu at (308.2, -406.2)
- added Q4: TPN22006NH,LQ, footprint:TPN22006NHLQ, F.Cu at (302.2, -339.0)
- added Q5: TPN22006NH,LQ, footprint:TPN22006NHLQ, F.Cu at (297.9, -406.2)
- added Q6: TPN22006NH,LQ, footprint:TPN22006NHLQ, F.Cu at (291.5, -339.0)
- added Q7: TPN22006NH,LQ, footprint:TPN22006NHLQ, F.Cu at (287.3, -406.3)
- added Q8: TPN22006NH,LQ, footprint:TPN22006NHLQ, F.Cu at (280.7, -339.0)
- added Q9: TPN22006NH,LQ, footprint:TPN22006NHLQ, F.Cu at (268.1, -406.2)
- added U5: 74HC244, footprint:SOP65P640X110-20N, F.Cu at (193.0, -368.9)
- J8: moved to B.Cu
- moved D3 573.9 mm to (314.8, -333.9), turned to 180 degrees
- moved D5 559.2 mm to (304.2, -334.3), turned to 180 degrees
- moved D7 544.8 mm to (293.4, -334.3), turned to 180 degrees
- moved D4 534.5 mm to (306.3, -410.9)
- moved U12 531.2 mm to (317.8, -341.1), turned to -90 degrees
- moved D9 530.4 mm to (282.7, -334.3), turned to 180 degrees
- moved D11 526.5 mm to (263.8, -334.2), turned to 180 degrees
- moved D6 521.2 mm to (295.9, -410.9)
- moved U14 517.9 mm to (307.2, -341.4), turned to -90 degrees
- moved D13 511.3 mm to (252.7, -334.1), turned to 180 degrees
- moved D8 507.8 mm to (285.4, -411.0)
- moved U16 504.6 mm to (296.5, -341.4), turned to -90 degrees
- moved R33 498.6 mm to (312.7, -343.3)
- moved R34 498.3 mm to (312.7, -341.6)
- moved D15 496.3 mm to (241.8, -334.2), turned to 180 degrees
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Routing:
- net /5V_4: track 0.00 -> 91.6 mm, vias 0 -> 22
- net /ENABLE: track 0.00 -> 61.0 mm, vias 0 -> 2
- net /LATCH: track 0.00 -> 60.1 mm, vias 0 -> 2
- net /CLK: track 0.00 -> 59.1 mm, vias 0 -> 2
- net /S8: track 0.00 -> 56.7 mm
- net /S16: track 0.00 -> 56.2 mm
- net /DATA_IN: track 0.00 -> 54.5 mm, vias 0 -> 2
- net /DATA1_OUT: track 0.00 -> 54.0 mm, vias 0 -> 2
- net /S6: track 0.00 -> 46.0 mm
- net /S14: track 0.00 -> 45.1 mm
- net /24V2_GND: track 0.00 -> 40.7 mm
- net /S9: track 0.00 -> 38.2 mm, vias 0 -> 2
- net /S1: track 0.00 -> 37.9 mm, vias 0 -> 2
- net /S12: track 0.00 -> 35.8 mm
- net /S4: track 0.00 -> 35.5 mm
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- added copper zone on B.Cu, net /24V2
- added copper zone on F.Cu, net /24V2
- added copper zone on F.Cu, net /24V2_GND
- added copper zone on B.Cu, net /5V_4
- added copper zone on F.Cu, net /5V_4
- added copper zone on B.Cu, net /GND_4
- added copper zone on F.Cu, net /SOL1-
- added copper zone on F.Cu, net /SOL10-
- added copper zone on F.Cu, net /SOL11-
- added copper zone on F.Cu, net /SOL12-
- added copper zone on F.Cu, net /SOL13-
- added copper zone on F.Cu, net /SOL14-
- added copper zone on F.Cu, net /SOL15-
- added copper zone on F.Cu, net /SOL16-
- added copper zone on F.Cu, net /SOL2-
- added copper zone on F.Cu, net /SOL3-
- added copper zone on F.Cu, net /SOL4-
- added copper zone on F.Cu, net /SOL5-
- added copper zone on F.Cu, net /SOL6-
- added copper zone on F.Cu, net /SOL7-
- added copper zone on F.Cu, net /SOL8-
- added copper zone on F.Cu, net /SOL9-
Other:
- outline, holes or cut-outs redrawn

Commit message: ,
,
Parts:
- added J32: SOL25, footprint:2PIN, F.Cu at (141.0, -424.8)
- added J33: SOL26, footprint:2PIN, F.Cu at (105.6, -425.2)
- added J34: SOL27, footprint:2PIN, F.Cu at (64.5, -426.2)
- added J35: SOL28, footprint:2PIN, F.Cu at (30.8, -429.4)
- added J36: SOL29, footprint:2PIN, F.Cu at (-79.1, -577.2)
- added J37: SOL30, footprint:2PIN, F.Cu at (-104.7, -569.9)
- added J38: SOL31, footprint:2PIN, F.Cu at (-98.3, -569.9)
- added J39: SOL32, footprint:2PIN, F.Cu at (-91.9, -569.9)
- added J40: SOL33, footprint:2PIN, F.Cu at (-70.8, -577.8)
- added J41: SOL34, footprint:2PIN, F.Cu at (-64.4, -577.8)
- added J42: SOL35, footprint:2PIN, F.Cu at (-58.0, -577.8)
- added J43: SOL36, footprint:2PIN, F.Cu at (-51.6, -577.8)
- added J44: SOL37, footprint:2PIN, F.Cu at (-70.8, -570.5)
- added J45: SOL38, footprint:2PIN, F.Cu at (-64.4, -570.5)
- added J46: SOL39, footprint:2PIN, F.Cu at (-58.0, -570.5)
- added J47: SOL40, footprint:2PIN, F.Cu at (-51.6, -570.5)
- added J48: SOL41, footprint:2PIN, F.Cu at (-70.8, -563.1)
- added J49: SOL42, footprint:2PIN, F.Cu at (-64.4, -563.1)
- added J50: SOL43, footprint:2PIN, F.Cu at (-58.0, -563.1)
- added J51: SOL44, footprint:2PIN, F.Cu at (-51.6, -563.1)
- added J52: SOL45, footprint:2PIN, F.Cu at (-70.8, -555.8)
- added J53: SOL46, footprint:2PIN, F.Cu at (-64.4, -555.8)
- added J54: SOL47, footprint:2PIN, F.Cu at (-58.0, -555.8)
- added J55: SOL48, footprint:2PIN, F.Cu at (-51.6, -555.8)
- added Q101: TPN22006NH,LQ, footprint:TPN22006NHLQ, F.Cu at (138.6, -411.0)
- added Q102: TPN22006NH,LQ, footprint:TPN22006NHLQ, F.Cu at (101.3, -411.4)
- added Q103: TPN22006NH,LQ, footprint:TPN22006NHLQ, F.Cu at (58.3, -412.4)
- added Q104: TPN22006NH,LQ, footprint:TPN22006NHLQ, F.Cu at (22.7, -415.6)
- added Q105: TPN22006NH,LQ, footprint:TPN22006NHLQ, F.Cu at (-89.1, -563.4)
- added Q106: TPN22006NH,LQ, footprint:TPN22006NHLQ, F.Cu at (-107.1, -558.1)
- added Q107: TPN22006NH,LQ, footprint:TPN22006NHLQ, F.Cu at (-102.6, -558.1)
- added Q108: TPN22006NH,LQ, footprint:TPN22006NHLQ, F.Cu at (-98.1, -558.1)
- added Q25: TPN22006NH,LQ, footprint:TPN22006NHLQ, F.Cu at (-47.6, -578.7)
- added Q26: TPN22006NH,LQ, footprint:TPN22006NHLQ, F.Cu at (-43.1, -578.7)
- added Q27: TPN22006NH,LQ, footprint:TPN22006NHLQ, F.Cu at (-38.6, -578.7)
- added Q28: TPN22006NH,LQ, footprint:TPN22006NHLQ, F.Cu at (-34.1, -578.7)
- added Q29: TPN22006NH,LQ, footprint:TPN22006NHLQ, F.Cu at (-47.6, -573.4)
- added Q30: TPN22006NH,LQ, footprint:TPN22006NHLQ, F.Cu at (-43.1, -573.4)
- added Q31: TPN22006NH,LQ, footprint:TPN22006NHLQ, F.Cu at (-38.6, -573.4)
- added Q32: TPN22006NH,LQ, footprint:TPN22006NHLQ, F.Cu at (-34.1, -573.4)
- added Q33: TPN22006NH,LQ, footprint:TPN22006NHLQ, F.Cu at (-47.6, -568.1)
- added Q34: TPN22006NH,LQ, footprint:TPN22006NHLQ, F.Cu at (-43.1, -568.1)
- added Q35: TPN22006NH,LQ, footprint:TPN22006NHLQ, F.Cu at (-38.6, -568.1)
- added Q36: TPN22006NH,LQ, footprint:TPN22006NHLQ, F.Cu at (-34.1, -568.1)
- added Q37: TPN22006NH,LQ, footprint:TPN22006NHLQ, F.Cu at (-47.6, -562.8)
- added Q38: TPN22006NH,LQ, footprint:TPN22006NHLQ, F.Cu at (-43.1, -562.8)
- added Q39: TPN22006NH,LQ, footprint:TPN22006NHLQ, F.Cu at (-38.6, -562.8)
- added Q40: TPN22006NH,LQ, footprint:TPN22006NHLQ, F.Cu at (-34.1, -562.8)
- added U101: 74HC244, footprint:SOP65P640X110-20N, F.Cu at (155.7, -488.0)
- J31: moved to B.Cu
- moved C10 379.0 mm to (187.2, -376.5), turned to 180 degrees
- moved C11 378.7 mm to (187.2, -374.6), turned to 180 degrees
- moved C12 376.4 mm to (187.3, -378.3)
- moved U47 373.6 mm to (192.6, -374.9), turned to -90 degrees
- moved U11 353.9 mm to (177.8, -487.6)
- moved Y1 351.5 mm to (170.0, -487.5), turned to -90 degrees
- moved C65 341.4 mm to (185.0, -489.1)
- moved C66 341.3 mm to (185.0, -487.1)
- moved C67 341.3 mm to (185.0, -485.1), turned to 180 degrees
- moved D101 337.2 mm to (123.1, -420.0)
- moved R55 328.1 mm to (184.9, -490.9), turned to 180 degrees
- moved C64 328.1 mm to (170.1, -483.0), turned to 180 degrees
- moved C63 327.1 mm to (170.3, -492.5)
- moved R52 322.2 mm to (178.3, -494.1)
- moved R60 316.8 mm to (175.1, -494.1)
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Routing:
- net /CLK: track 59.1 -> 5.71 mm, vias 2 -> 1
- net /LATCH: track 60.1 -> 7.52 mm, vias 2 -> 1
- net /ENABLE: track 61.0 -> 11.4 mm, vias 2 -> 1
- net /DATA_IN: track 54.5 -> 6.79 mm, vias 2 -> 0
- net /DATA1_OUT: track 54.0 -> 6.45 mm, vias 2 -> 1
- net /S17: track 0.00 -> 44.6 mm, vias 0 -> 2
- net /S23: track 0.00 -> 42.1 mm
- net /S20: track 0.00 -> 31.6 mm
- net /S22: track 0.00 -> 31.3 mm
- net /S24: track 0.00 -> 31.2 mm
- net /S19: track 0.00 -> 31.1 mm
- net /GND_4: track 14.4 -> 42.1 mm, vias 2 -> 5
- net /24V2_GND: track 40.7 -> 14.3 mm
- net Net-(R9-Pad1): track 0.00 -> 17.0 mm
- net /24V2: track 23.1 -> 39.8 mm, vias 34 -> 42
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- added copper zone on F.Cu, net /SOL17-
- added copper zone on F.Cu, net /SOL18-
- added copper zone on F.Cu, net /SOL19-
- added copper zone on F.Cu, net /SOL20-
- added copper zone on F.Cu, net /SOL21-
- added copper zone on F.Cu, net /SOL22-
- added copper zone on F.Cu, net /SOL23-
- added copper zone on F.Cu, net /SOL24-
Other:
- outline, holes or cut-outs redrawn

Commit message: .
.
Parts:
- removed the D27 at (-183.7, -564.2)
- removed the D41 at (-166.9, -597.5)
- removed the J41 at (-64.4, -577.8)
- removed the J55 at (-51.6, -555.8)
- removed the Q26 at (-43.1, -578.7)
- removed the Q40 at (-34.1, -562.8)
- removed the R139 at (-128.7, -536.7)
- removed the R148 at (-128.7, -514.1)
- removed the R149 at (-128.7, -511.6)
- removed the R177 at (-124.7, -506.6)
- removed the R192 at (-120.6, -514.1)
- removed the R193 at (-120.6, -511.6)
- removed the U57 at (-138.6, -594.0)
- removed the U80 at (-129.0, -585.8)
- added C27: 0.1uF, Capacitor_SMD:C_0603_1608Metric, F.Cu at (64.0, 30.2)
- added C28: 1uF, Capacitor_SMD:C_0603_1608Metric, F.Cu at (64.0, 32.7)
- added C29: 10uF, Capacitor_SMD:C_0603_1608Metric, F.Cu at (64.0, 35.2)
- added C30: 0.1uF, Capacitor_SMD:C_0603_1608Metric, F.Cu at (64.0, 37.7)
- added C31: 1uF, Capacitor_SMD:C_0603_1608Metric, F.Cu at (64.0, 40.2)
- added C32: 10uF, Capacitor_SMD:C_0603_1608Metric, F.Cu at (64.0, 42.7)
- added C33: 0.1uF, Capacitor_SMD:C_0603_1608Metric, F.Cu at (64.0, 45.2)
- added C34: 1uF, Capacitor_SMD:C_0603_1608Metric, F.Cu at (64.0, 47.7)
- added C35: 10uF, Capacitor_SMD:C_0603_1608Metric, F.Cu at (64.0, 50.2)
- added C38: 0.1uF, Capacitor_SMD:C_0603_1608Metric, F.Cu at (64.0, 52.7)
- added C39: 1uF, Capacitor_SMD:C_0603_1608Metric, F.Cu at (64.0, 55.3)
- added C43: 10uF, Capacitor_SMD:C_0603_1608Metric, F.Cu at (64.0, 57.8)
- added D27: DIODE, Diode_SMD:D_SMB, F.Cu at (156.1, -330.5)
- added D27: DIODE, Diode_SMD:D_SMB, F.Cu at (3.72, 31.7)
- added D41: DIODE, Diode_SMD:D_SMB, F.Cu at (86.0, -330.6)
- added D41: DIODE, Diode_SMD:D_SMB, F.Cu at (3.72, 37.2)
- added D42: DIODE, Diode_SMD:D_SMB, F.Cu at (3.72, 42.8)
- added D43: DIODE, Diode_SMD:D_SMB, F.Cu at (3.72, 48.3)
- added D44: DIODE, Diode_SMD:D_SMB, F.Cu at (3.72, 53.9)
- added D45: DIODE, Diode_SMD:D_SMB, F.Cu at (3.72, 59.4)
- added D46: DIODE, Diode_SMD:D_SMB, F.Cu at (3.72, 65.0)
- added D47: DIODE, Diode_SMD:D_SMB, F.Cu at (12.1, 31.7)
- added D48: DIODE, Diode_SMD:D_SMB, F.Cu at (12.1, 37.2)
- added D49: DIODE, Diode_SMD:D_SMB, F.Cu at (12.1, 42.8)
- added D50: DIODE, Diode_SMD:D_SMB, F.Cu at (12.1, 48.3)
- added D51: DIODE, Diode_SMD:D_SMB, F.Cu at (12.1, 53.9)
- added D52: DIODE, Diode_SMD:D_SMB, F.Cu at (12.1, 59.4)
- added D53: DIODE, Diode_SMD:D_SMB, F.Cu at (12.1, 65.0)
- added D54: DIODE, Diode_SMD:D_SMB, F.Cu at (20.5, 31.7)
- added D55: DIODE, Diode_SMD:D_SMB, F.Cu at (20.5, 37.2)
- added D56: DIODE, Diode_SMD:D_SMB, F.Cu at (20.5, 42.8)
- added D57: DIODE, Diode_SMD:D_SMB, F.Cu at (20.5, 48.3)
- added D58: DIODE, Diode_SMD:D_SMB, F.Cu at (20.5, 53.9)
- added D59: DIODE, Diode_SMD:D_SMB, F.Cu at (20.5, 59.4)
- added D60: DIODE, Diode_SMD:D_SMB, F.Cu at (20.5, 65.0)
- added D61: DIODE, Diode_SMD:D_SMB, F.Cu at (28.9, 31.7)
- added D62: DIODE, Diode_SMD:D_SMB, F.Cu at (28.9, 37.2)
- added D63: DIODE, Diode_SMD:D_SMB, F.Cu at (28.9, 42.8)
- added D64: DIODE, Diode_SMD:D_SMB, F.Cu at (28.9, 48.3)
- added D65: DIODE, Diode_SMD:D_SMB, F.Cu at (28.9, 53.9)
- added J41: SOL34, footprint:2PIN, F.Cu at (4.12, 2.88)
- added J41: SOL34, footprint:2PIN, B.Cu at (157.1, -322.9)
- added J55: SOL48, footprint:2PIN, F.Cu at (10.5, 2.88)
- added J55: SOL48, footprint:2PIN, B.Cu at (87.1, -322.9)
- added J58: SOL25, footprint:2PIN, F.Cu at (16.9, 2.88)
- added J59: SOL26, footprint:2PIN, F.Cu at (23.3, 2.88)
- added J60: SOL27, footprint:2PIN, F.Cu at (29.7, 2.88)
- added J61: SOL28, footprint:2PIN, F.Cu at (36.1, 2.88)
- added J62: SOL29, footprint:2PIN, F.Cu at (42.5, 2.88)
- added J63: SOL30, footprint:2PIN, F.Cu at (4.12, 10.2)
- added J64: SOL31, footprint:2PIN, F.Cu at (10.5, 10.2)
- added J65: SOL32, footprint:2PIN, F.Cu at (16.9, 10.2)
- added J66: SOL35, footprint:2PIN, F.Cu at (23.3, 10.2)
- added J67: SOL38, footprint:2PIN, F.Cu at (29.7, 10.2)
- added J68: SOL34, footprint:2PIN, F.Cu at (36.1, 10.2)
- added J69: SOL37, footprint:2PIN, F.Cu at (42.5, 10.2)
- added J70: SOL33, footprint:2PIN, F.Cu at (4.12, 17.6)
- added J71: SOL36, footprint:2PIN, F.Cu at (10.5, 17.6)
- added J72: SOL39, footprint:2PIN, F.Cu at (16.9, 17.6)
- added J73: SOL40, footprint:2PIN, F.Cu at (23.3, 17.6)
- added J74: SOL44, footprint:2PIN, F.Cu at (29.7, 17.6)
- added J75: SOL47, footprint:2PIN, F.Cu at (36.1, 17.6)
- added J76: SOL41, footprint:2PIN, F.Cu at (42.5, 17.6)
- added J77: SOL42, footprint:2PIN, F.Cu at (4.12, 24.9)
- added J78: SOL43, footprint:2PIN, F.Cu at (10.5, 24.9)
- added J79: SOL45, footprint:2PIN, F.Cu at (16.9, 24.9)
- added J80: SOL46, footprint:2PIN, F.Cu at (23.3, 24.9)
- added J81: SOL48, footprint:2PIN, F.Cu at (29.7, 24.9)
- added J82: SHIFT_DATA_TOSS, footprint:SHIFT_DATA_TOSS, F.Cu at (45.3, 22.7)
- added Q26: TPN22006NH,LQ, footprint:TPN22006NHLQ, F.Cu at (46.5, 1.95)
- added Q26: TPN22006NH,LQ, footprint:TPN22006NHLQ, F.Cu at (154.6, -336.6)
- added Q40: TPN22006NH,LQ, footprint:TPN22006NHLQ, F.Cu at (84.6, -336.7)
- added Q40: TPN22006NH,LQ, footprint:TPN22006NHLQ, F.Cu at (51.0, 1.95)
- added Q41: TPN22006NH,LQ, footprint:TPN22006NHLQ, F.Cu at (55.5, 1.95)
- added Q42: TPN22006NH,LQ, footprint:TPN22006NHLQ, F.Cu at (60.0, 1.95)
- added Q43: TPN22006NH,LQ, footprint:TPN22006NHLQ, F.Cu at (64.5, 1.95)
- added Q44: TPN22006NH,LQ, footprint:TPN22006NHLQ, F.Cu at (69.0, 1.95)
- added Q45: TPN22006NH,LQ, footprint:TPN22006NHLQ, F.Cu at (73.5, 1.95)
- added Q46: TPN22006NH,LQ, footprint:TPN22006NHLQ, F.Cu at (46.5, 7.25)
- added Q47: TPN22006NH,LQ, footprint:TPN22006NHLQ, F.Cu at (51.0, 7.25)
- added Q48: TPN22006NH,LQ, footprint:TPN22006NHLQ, F.Cu at (55.5, 7.25)
- added Q49: TPN22006NH,LQ, footprint:TPN22006NHLQ, F.Cu at (60.0, 7.25)
- added Q50: TPN22006NH,LQ, footprint:TPN22006NHLQ, F.Cu at (64.5, 7.25)
- added Q51: TPN22006NH,LQ, footprint:TPN22006NHLQ, F.Cu at (69.0, 7.25)
- added Q52: TPN22006NH,LQ, footprint:TPN22006NHLQ, F.Cu at (73.5, 7.25)
- added Q53: TPN22006NH,LQ, footprint:TPN22006NHLQ, F.Cu at (46.5, 12.6)
- added Q54: TPN22006NH,LQ, footprint:TPN22006NHLQ, F.Cu at (51.0, 12.6)
- added Q55: TPN22006NH,LQ, footprint:TPN22006NHLQ, F.Cu at (55.5, 12.6)
- added Q56: TPN22006NH,LQ, footprint:TPN22006NHLQ, F.Cu at (60.0, 12.6)
- added Q57: TPN22006NH,LQ, footprint:TPN22006NHLQ, F.Cu at (64.5, 12.6)
- added Q58: TPN22006NH,LQ, footprint:TPN22006NHLQ, F.Cu at (69.0, 12.6)
- added Q59: TPN22006NH,LQ, footprint:TPN22006NHLQ, F.Cu at (73.5, 12.6)
- added Q60: TPN22006NH,LQ, footprint:TPN22006NHLQ, F.Cu at (46.5, 17.9)
- added Q61: TPN22006NH,LQ, footprint:TPN22006NHLQ, F.Cu at (51.0, 17.9)
- added Q62: TPN22006NH,LQ, footprint:TPN22006NHLQ, F.Cu at (55.5, 17.9)
- added Q63: TPN22006NH,LQ, footprint:TPN22006NHLQ, F.Cu at (60.0, 17.9)
- added Q64: TPN22006NH,LQ, footprint:TPN22006NHLQ, F.Cu at (64.5, 17.9)
- added R100: 22kΩ, Resistor_SMD:R_0603_1608Metric, F.Cu at (72.1, 37.7)
- added R101: 22kΩ, Resistor_SMD:R_0603_1608Metric, F.Cu at (72.1, 40.2)
- added R102: 22kΩ, Resistor_SMD:R_0603_1608Metric, F.Cu at (72.1, 42.7)
- added R103: 22kΩ, Resistor_SMD:R_0603_1608Metric, F.Cu at (72.1, 45.2)
- added R104: 22kΩ, Resistor_SMD:R_0603_1608Metric, F.Cu at (72.1, 47.7)
- added R130: 22kΩ, Resistor_SMD:R_0603_1608Metric, F.Cu at (72.1, 50.2)
- added R131: 3.3kΩ, Resistor_SMD:R_0603_1608Metric, F.Cu at (72.1, 52.7)
- added R132: 3.3kΩ, Resistor_SMD:R_0603_1608Metric, F.Cu at (72.1, 55.3)
- added R133: 3.3kΩ, Resistor_SMD:R_0603_1608Metric, F.Cu at (72.1, 57.8)
- added R134: 3.3kΩ, Resistor_SMD:R_0603_1608Metric, F.Cu at (72.1, 60.3)
- added R135: 3.3kΩ, Resistor_SMD:R_0603_1608Metric, F.Cu at (72.1, 62.8)
- added R136: 3.3kΩ, Resistor_SMD:R_0603_1608Metric, F.Cu at (76.1, 30.2)
- added R137: 3.3kΩ, Resistor_SMD:R_0603_1608Metric, F.Cu at (76.1, 32.7)
- added R139: 3.3kΩ, Resistor_SMD:R_0603_1608Metric, F.Cu at (155.5, -343.2)
- added R139: 3.3kΩ, Resistor_SMD:R_0603_1608Metric, F.Cu at (76.1, 35.2)
- added R148: 22kΩ, Resistor_SMD:R_0603_1608Metric, F.Cu at (76.1, 37.7)
- added R148: 22kΩ, Resistor_SMD:R_0603_1608Metric, F.Cu at (155.6, -341.4)
- added R149: 22kΩ, Resistor_SMD:R_0603_1608Metric, F.Cu at (76.1, 40.2)
- added R149: 22kΩ, Resistor_SMD:R_0603_1608Metric, F.Cu at (155.6, -339.6)
- added R162: 3.3kΩ, Resistor_SMD:R_0603_1608Metric, F.Cu at (76.1, 42.7)
- added R163: 22kΩ, Resistor_SMD:R_0603_1608Metric, F.Cu at (76.1, 45.2)
- added R164: 22kΩ, Resistor_SMD:R_0603_1608Metric, F.Cu at (76.1, 47.7)
- added R165: 22kΩ, Resistor_SMD:R_0603_1608Metric, F.Cu at (76.1, 50.2)
- added R166: 22kΩ, Resistor_SMD:R_0603_1608Metric, F.Cu at (76.1, 52.7)
- added R167: 22kΩ, Resistor_SMD:R_0603_1608Metric, F.Cu at (76.1, 55.3)
- added R168: 22kΩ, Resistor_SMD:R_0603_1608Metric, F.Cu at (76.1, 57.8)
- added R169: 22kΩ, Resistor_SMD:R_0603_1608Metric, F.Cu at (76.1, 60.3)
- added R177: 3.3kΩ, Resistor_SMD:R_0603_1608Metric, F.Cu at (85.5, -343.2)
- added R177: 3.3kΩ, Resistor_SMD:R_0603_1608Metric, F.Cu at (76.1, 62.8)
- added R192: 22kΩ, Resistor_SMD:R_0603_1608Metric, F.Cu at (80.1, 30.2)
- added R192: 22kΩ, Resistor_SMD:R_0603_1608Metric, F.Cu at (85.5, -341.5)
- added R193: 22kΩ, Resistor_SMD:R_0603_1608Metric, F.Cu at (80.1, 32.7)
- added R193: 22kΩ, Resistor_SMD:R_0603_1608Metric, F.Cu at (85.5, -339.7)
- added R194: 22kΩ, Resistor_SMD:R_0603_1608Metric, F.Cu at (80.1, 35.2)
- added R195: 22kΩ, Resistor_SMD:R_0603_1608Metric, F.Cu at (80.1, 37.7)
- added R196: 22kΩ, Resistor_SMD:R_0603_1608Metric, F.Cu at (80.1, 40.2)
- added R197: 22kΩ, Resistor_SMD:R_0603_1608Metric, F.Cu at (80.1, 42.7)
- added R198: 22kΩ, Resistor_SMD:R_0603_1608Metric, F.Cu at (80.1, 45.2)
- added R199: 22kΩ, Resistor_SMD:R_0603_1608Metric, F.Cu at (80.1, 47.7)
- added R200: 22kΩ, Resistor_SMD:R_0603_1608Metric, F.Cu at (80.1, 50.2)
- added R201: 22kΩ, Resistor_SMD:R_0603_1608Metric, F.Cu at (80.1, 52.7)
- added R202: 22kΩ, Resistor_SMD:R_0603_1608Metric, F.Cu at (80.1, 55.3)
- added R203: 3.3kΩ, Resistor_SMD:R_0603_1608Metric, F.Cu at (80.1, 57.8)
- added R204: 3.3kΩ, Resistor_SMD:R_0603_1608Metric, F.Cu at (80.1, 60.3)
- added R205: 3.3kΩ, Resistor_SMD:R_0603_1608Metric, F.Cu at (80.1, 62.8)
- added R206: 3.3kΩ, Resistor_SMD:R_0603_1608Metric, F.Cu at (84.1, 30.2)
- added R207: 3.3kΩ, Resistor_SMD:R_0603_1608Metric, F.Cu at (84.1, 32.7)
- added R208: 3.3kΩ, Resistor_SMD:R_0603_1608Metric, F.Cu at (84.1, 35.2)
- added R209: 3.3kΩ, Resistor_SMD:R_0603_1608Metric, F.Cu at (84.1, 37.7)
- added R210: 3.3kΩ, Resistor_SMD:R_0603_1608Metric, F.Cu at (84.1, 40.2)
- added R211: 22kΩ, Resistor_SMD:R_0603_1608Metric, F.Cu at (84.1, 42.7)
- added R212: 22kΩ, Resistor_SMD:R_0603_1608Metric, F.Cu at (84.1, 45.2)
- added R213: 22kΩ, Resistor_SMD:R_0603_1608Metric, F.Cu at (84.1, 47.7)
- added R214: 22kΩ, Resistor_SMD:R_0603_1608Metric, F.Cu at (84.1, 50.2)
- added R215: 22kΩ, Resistor_SMD:R_0603_1608Metric, F.Cu at (84.1, 52.7)
- added R216: 22kΩ, Resistor_SMD:R_0603_1608Metric, F.Cu at (84.1, 55.3)
- added R217: 22kΩ, Resistor_SMD:R_0603_1608Metric, F.Cu at (84.1, 57.8)
- added R218: 22kΩ, Resistor_SMD:R_0603_1608Metric, F.Cu at (84.1, 60.3)
- added R219: 22kΩ, Resistor_SMD:R_0603_1608Metric, F.Cu at (84.1, 62.8)
- added R220: 22kΩ, Resistor_SMD:R_0603_1608Metric, F.Cu at (88.1, 30.2)
- added R221: 22kΩ, Resistor_SMD:R_0603_1608Metric, F.Cu at (88.1, 32.7)
- added R222: 22kΩ, Resistor_SMD:R_0603_1608Metric, F.Cu at (88.1, 35.2)
- added R223: 22kΩ, Resistor_SMD:R_0603_1608Metric, F.Cu at (88.1, 37.7)
- added R224: 22kΩ, Resistor_SMD:R_0603_1608Metric, F.Cu at (88.1, 40.2)
- added R225: 22kΩ, Resistor_SMD:R_0603_1608Metric, F.Cu at (88.1, 42.7)
- added R226: 22kΩ, Resistor_SMD:R_0603_1608Metric, F.Cu at (88.1, 45.2)
- added R80: 100Ω, Resistor_SMD:R_0603_1608Metric, F.Cu at (64.0, 60.3)
- added R81: 3.3kΩ, Resistor_SMD:R_0603_1608Metric, F.Cu at (64.0, 62.8)
- added R82: 3.3kΩ, Resistor_SMD:R_0603_1608Metric, F.Cu at (68.0, 30.2)
- added R83: 3.3kΩ, Resistor_SMD:R_0603_1608Metric, F.Cu at (68.0, 32.7)
- added R84: 3.3kΩ, Resistor_SMD:R_0603_1608Metric, F.Cu at (68.0, 35.2)
- added R85: 3.3kΩ, Resistor_SMD:R_0603_1608Metric, F.Cu at (68.0, 37.7)
- added R86: 3.3kΩ, Resistor_SMD:R_0603_1608Metric, F.Cu at (68.0, 40.2)
- added R87: 3.3kΩ, Resistor_SMD:R_0603_1608Metric, F.Cu at (68.0, 42.7)
- added R88: 3.3kΩ, Resistor_SMD:R_0603_1608Metric, F.Cu at (68.0, 45.2)
- added R89: 22kΩ, Resistor_SMD:R_0603_1608Metric, F.Cu at (68.0, 47.7)
- added R90: 22kΩ, Resistor_SMD:R_0603_1608Metric, F.Cu at (68.0, 50.2)
- added R91: 22kΩ, Resistor_SMD:R_0603_1608Metric, F.Cu at (68.0, 52.7)
- added R92: 22kΩ, Resistor_SMD:R_0603_1608Metric, F.Cu at (68.0, 55.3)
- added R93: 22kΩ, Resistor_SMD:R_0603_1608Metric, F.Cu at (68.0, 57.8)
- added R94: 22kΩ, Resistor_SMD:R_0603_1608Metric, F.Cu at (68.0, 60.3)
- added R95: 22kΩ, Resistor_SMD:R_0603_1608Metric, F.Cu at (68.0, 62.8)
- added R97: 22kΩ, Resistor_SMD:R_0603_1608Metric, F.Cu at (72.1, 30.2)
- added R98: 22kΩ, Resistor_SMD:R_0603_1608Metric, F.Cu at (72.1, 32.7)
- added R99: 22kΩ, Resistor_SMD:R_0603_1608Metric, F.Cu at (72.1, 35.2)
- added U19: 74HC244, footprint:SOP65P640X110-20N, F.Cu at (69.8, 24.8)
- added U20: TLP291, Package_SO:SOIC-4_4.55x2.6mm_P1.27mm, F.Cu at (37.9, 31.0)
- added U21: TLP291, Package_SO:SOIC-4_4.55x2.6mm_P1.27mm, F.Cu at (37.9, 35.1)
- added U22: TLP291, Package_SO:SOIC-4_4.55x2.6mm_P1.27mm, F.Cu at (37.9, 39.3)
- added U23: TLP291, Package_SO:SOIC-4_4.55x2.6mm_P1.27mm, F.Cu at (37.9, 43.4)
- added U24: TLP291, Package_SO:SOIC-4_4.55x2.6mm_P1.27mm, F.Cu at (37.9, 47.6)
- added U25: TLP291, Package_SO:SOIC-4_4.55x2.6mm_P1.27mm, F.Cu at (37.9, 51.7)
- added U26: TLP291, Package_SO:SOIC-4_4.55x2.6mm_P1.27mm, F.Cu at (37.9, 55.9)
- added U35: TLP291, Package_SO:SOIC-4_4.55x2.6mm_P1.27mm, F.Cu at (37.9, 60.0)
- added U36: 74HCT595, Package_SO:SSOP-16_5.3x6.2mm_P0.65mm, F.Cu at (80.9, 3.38)
- added U37: TLP291, Package_SO:SOIC-4_4.55x2.6mm_P1.27mm, F.Cu at (37.9, 64.2)
- added U38: TLP291, Package_SO:SOIC-4_4.55x2.6mm_P1.27mm, F.Cu at (47.6, 31.0)
- added U39: TLP291, Package_SO:SOIC-4_4.55x2.6mm_P1.27mm, F.Cu at (47.6, 35.1)
- added U4: ISP, footprint:TPN22006NHLQ, F.Cu at (183.2, -496.8)
- added U40: TLP291, Package_SO:SOIC-4_4.55x2.6mm_P1.27mm, F.Cu at (47.6, 39.3)
- added U41: TLP291, Package_SO:SOIC-4_4.55x2.6mm_P1.27mm, F.Cu at (47.6, 43.4)
- added U42: TLP291, Package_SO:SOIC-4_4.55x2.6mm_P1.27mm, F.Cu at (47.6, 47.6)
- added U48: TLP291, Package_SO:SOIC-4_4.55x2.6mm_P1.27mm, F.Cu at (47.6, 51.7)
- added U49: TLP291, Package_SO:SOIC-4_4.55x2.6mm_P1.27mm, F.Cu at (47.6, 55.9)
- added U50: 74HCT595, Package_SO:SSOP-16_5.3x6.2mm_P0.65mm, F.Cu at (80.9, 11.1)
- added U51: TLP291, Package_SO:SOIC-4_4.55x2.6mm_P1.27mm, F.Cu at (47.6, 60.0)
- added U52: TLP291, Package_SO:SOIC-4_4.55x2.6mm_P1.27mm, F.Cu at (47.6, 64.2)
- added U53: TLP291, Package_SO:SOIC-4_4.55x2.6mm_P1.27mm, F.Cu at (57.2, 31.0)
- added U54: TLP291, Package_SO:SOIC-4_4.55x2.6mm_P1.27mm, F.Cu at (57.2, 35.1)
- added U55: TLP291, Package_SO:SOIC-4_4.55x2.6mm_P1.27mm, F.Cu at (57.2, 39.3)
- added U57: TLP291, Package_SO:SOIC-4_4.55x2.6mm_P1.27mm, F.Cu at (57.2, 43.4)
- added U57: TLP291, Package_SO:SOIC-4_4.55x2.6mm_P1.27mm, F.Cu at (155.6, -348.5)
- added U65: TLP291, Package_SO:SOIC-4_4.55x2.6mm_P1.27mm, F.Cu at (57.2, 47.6)
- added U66: TLP291, Package_SO:SOIC-4_4.55x2.6mm_P1.27mm, F.Cu at (57.2, 51.7)
- added U67: TLP291, Package_SO:SOIC-4_4.55x2.6mm_P1.27mm, F.Cu at (57.2, 55.9)
- added U68: 74HCT595, Package_SO:SSOP-16_5.3x6.2mm_P0.65mm, F.Cu at (80.9, 18.9)
- added U80: TLP291, Package_SO:SOIC-4_4.55x2.6mm_P1.27mm, F.Cu at (85.7, -348.6)
- added U80: TLP291, Package_SO:SOIC-4_4.55x2.6mm_P1.27mm, F.Cu at (57.2, 60.0)
- J32, J33, J34, J35, J36, J37, J38, J39, J40, J42, J43, J44, J45, J46, J47, J48, J49, J50, J51, J52, J53, J54: moved to B.Cu
- moved D106 415.1 mm to (176.1, -330.4), turned to -90 degrees
- moved D31 410.2 mm to (136.1, -330.6), turned to -90 degrees
- moved D108 400.5 mm to (166.1, -330.6), turned to -90 degrees
- moved D29 398.0 mm to (146.2, -330.5), turned to -90 degrees
- moved D33 395.4 mm to (126.1, -330.5), turned to -90 degrees
- moved D35 380.5 mm to (116.1, -330.6), turned to -90 degrees
- moved D105 376.8 mm to (175.4, -412.3), turned to 90 degrees
- moved J37 374.8 mm to (177.1, -322.9)
- moved C16 374.2 mm to (184.1, -366.5), turned to 180 degrees
- moved C17 373.8 mm to (184.1, -364.8), turned to 180 degrees
- moved D26 373.8 mm to (155.4, -412.4), turned to 90 degrees
- moved C19 373.5 mm to (184.1, -363.1)
- moved U108 371.3 mm to (175.8, -348.8), turned to -90 degrees
- moved U59 370.3 mm to (145.6, -348.4), turned to -90 degrees
- moved R111 366.7 mm to (175.7, -343.4), turned to 180 degrees
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Routing:
- net /24V2: track 39.8 -> 99.7 mm, vias 42 -> 67
- net /S48: track 0.00 -> 55.2 mm
- net /S40: track 0.00 -> 54.5 mm
- net /S32: track 0.00 -> 54.0 mm
- net /CLK: track 5.71 -> 52.8 mm, vias 1 -> 2
- net /LATCH: track 7.52 -> 54.5 mm, vias 1 -> 2
- net /S46: track 0.00 -> 46.9 mm
- net /S38: track 0.00 -> 45.6 mm
- net /S30: track 0.00 -> 45.5 mm
- net /S41: track 0.00 -> 44.5 mm, vias 0 -> 2
- net /ENABLE: track 11.4 -> 55.7 mm, vias 1 -> 2
- net /S33: track 0.00 -> 44.0 mm, vias 0 -> 2
- net /S25: track 0.00 -> 42.8 mm, vias 0 -> 2
- net /DATA1_OUT: track 6.45 -> 48.0 mm, vias 1 -> 2
- net /S28: track 0.00 -> 38.6 mm
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- added copper zone on F.Cu, net /SOL25-
- added copper zone on F.Cu, net /SOL26-
- added copper zone on F.Cu, net /SOL27-
- added copper zone on F.Cu, net /SOL28-
- added copper zone on F.Cu, net /SOL29-
- added copper zone on F.Cu, net /SOL30-
- added copper zone on F.Cu, net /SOL31-
- added copper zone on F.Cu, net /SOL32-
- added copper zone on F.Cu, net /SOL33-
- added copper zone on F.Cu, net /SOL34-
- added copper zone on F.Cu, net /SOL35-
- added copper zone on F.Cu, net /SOL36-
- added copper zone on F.Cu, net /SOL37-
- added copper zone on F.Cu, net /SOL38-
- added copper zone on F.Cu, net /SOL39-
- added copper zone on F.Cu, net /SOL40-
- added copper zone on F.Cu, net /SOL41-
- added copper zone on F.Cu, net /SOL42-
- added copper zone on F.Cu, net /SOL43-
- added copper zone on F.Cu, net /SOL44-
- added copper zone on F.Cu, net /SOL45-
- added copper zone on F.Cu, net /SOL46-
- added copper zone on F.Cu, net /SOL47-
- added copper zone on F.Cu, net /SOL48-

Commit message: .
.
Parts:
- removed C13, C27, C30, C33, C36, C38, C40, C42, C45: 0.1uF, Capacitor_SMD:C_0603_1608Metric
- removed C14, C28, C31, C34, C39, C48, C58: 1uF, Capacitor_SMD:C_0603_1608Metric
- removed C15, C29, C32, C35, C43, C44, C60, C62: 10uF, Capacitor_SMD:C_0603_1608Metric
- removed C37: NC, Capacitor_SMD:C_0603_1608Metric
- removed C49, C53, C57: 22uF, Capacitor_SMD:C_0805_2012Metric
- removed D2: JD, Diode_SMD:D_SMB
- removed the D27 at (3.72, 31.7)
- removed the D41 at (3.72, 37.2)
- removed D42, D43, D44, D45, D46, D47, D48, D49, D50, D51, D52, D53, D54, D55, D56, D57, D58, D59, D60, D61, D62, D63, D64, D65: DIODE, Diode_SMD:D_SMB
- removed the J41 at (4.12, 2.88)
- removed the J55 at (10.5, 2.88)
- removed J58: SOL25, footprint:2PIN
- removed J59: SOL26, footprint:2PIN
- removed J60: SOL27, footprint:2PIN
- removed J61: SOL28, footprint:2PIN
- removed J62: SOL29, footprint:2PIN
- removed J63: SOL30, footprint:2PIN
- removed J64: SOL31, footprint:2PIN
- removed J65: SOL32, footprint:2PIN
- removed J66: SOL35, footprint:2PIN
- removed J67: SOL38, footprint:2PIN
- removed J68: SOL34, footprint:2PIN
- removed J69: SOL37, footprint:2PIN
- removed J70: SOL33, footprint:2PIN
- removed J71: SOL36, footprint:2PIN
- removed J72: SOL39, footprint:2PIN
- removed J73: SOL40, footprint:2PIN
- removed J74: SOL44, footprint:2PIN
- removed J75: SOL47, footprint:2PIN
- removed J76: SOL41, footprint:2PIN
- removed J77: SOL42, footprint:2PIN
- removed J78: SOL43, footprint:2PIN
- removed J79: SOL45, footprint:2PIN
- removed J80: SOL46, footprint:2PIN
- removed J81: SOL48, footprint:2PIN
- removed J82: SHIFT_DATA_TOSS, footprint:SHIFT_DATA_TOSS
- removed the Q26 at (46.5, 1.95)
- removed the Q40 at (51.0, 1.95)
- removed Q41, Q42, Q43, Q44, Q45, Q46, Q47, Q48, Q49, Q50, Q51, Q52, Q53, Q54, Q55, Q56, Q57, Q58, Q59, Q60, Q61, Q62, Q63, Q64: TPN22006NH,LQ, footprint:TPN22006NHLQ
- removed R100, R101, R102, R103, R104, R130, R131, R132, R133, R134, R135, R136, R137, R162, R163, R164, R165, R166, R167, R168, R169, R194, R195, R196, R197, R198, R199, R200, R201, R81, R82, R83, R84, R85, R86, R87, R88, R89, R90, R91, R92, R93, R94, R95, R97, R98, R99: 1kΩ, Resistor_SMD:R_0805_2012Metric
- removed R100, R101, R102, R103, R104, R130, R163, R164, R165, R166, R167, R168, R169, R194, R195, R196, R197, R198, R199, R200, R201, R202, R211, R212, R213, R214, R215, R216, R217, R218, R219, R220, R221, R222, R223, R224, R225, R226, R89, R90, R91, R92, R93, R94, R95, R97, R98, R99: 22kΩ, Resistor_SMD:R_0603_1608Metric
- removed R105, R80: 100Ω, Resistor_SMD:R_0603_1608Metric
- removed R131, R132, R133, R134, R135, R136, R137, R162, R203, R204, R205, R206, R207, R208, R209, R210, R81, R82, R83, R84, R85, R86, R87, R88: 3.3kΩ, Resistor_SMD:R_0603_1608Metric
- removed the R139 at (76.1, 35.2)
- removed the R148 at (76.1, 37.7)
- removed the R149 at (76.1, 40.2)
- removed the R177 at (76.1, 62.8)
- removed the R192 at (80.1, 30.2)
- removed the R193 at (80.1, 32.7)
- removed R44, R46: 1kΩ, Resistor_SMD:R_0603_1608Metric
- removed R45: 150Ω, Resistor_SMD:R_0603_1608Metric
- removed R53: 2kΩ, Resistor_SMD:R_0603_1608Metric
- removed U10: AP2127K-3.3, Package_TO_SOT_SMD:SOT-23-5
- removed U19: 74HC244, footprint:SOP65P640X110-20N
- removed U20, U21, U22, U23, U24, U25, U26, U35, U37, U38, U39, U40, U41, U42, U48, U49, U51, U52, U53, U54, U55, U65, U66, U67: TLP291, Package_SO:SOIC-4_4.55x2.6mm_P1.27mm
- removed U36, U50, U68: 74HCT595, Package_SO:SSOP-16_5.3x6.2mm_P0.65mm
- removed the U57 at (57.2, 43.4)
- removed the U80 at (57.2, 60.0)
- moved J8 721.8 mm to (-384.9, -241.0), turned to 0 degrees
- moved D1 720.2 mm to (-385.9, -248.5), turned to -90 degrees
- moved Q1 720.0 mm to (-387.2, -254.5), turned to 180 degrees
- moved R43 716.9 mm to (-386.2, -257.7), turned to 0 degrees
- moved R42 716.2 mm to (-386.2, -259.4), turned to 0 degrees
- moved R27 715.4 mm to (-386.2, -261.1), turned to 180 degrees
- moved U3 713.6 mm to (-386.3, -266.5), turned to -90 degrees
- moved J9 705.0 mm to (-387.7, -338.2), turned to 180 degrees
- moved U12 703.0 mm to (-386.3, -312.9), turned to 90 degrees
- moved D3 702.8 mm to (-386.7, -330.7), turned to 90 degrees
- moved J10 702.4 mm to (-374.9, -241.0), turned to 0 degrees
- moved R21 702.4 mm to (-386.3, -318.2), turned to 0 degrees
- moved R33 702.3 mm to (-386.3, -319.9), turned to 180 degrees
- moved R34 702.1 mm to (-386.2, -321.6), turned to 180 degrees
- moved D4 700.7 mm to (-375.9, -248.6), turned to -90 degrees
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Other:
- board size 345 x 346 mm -> 730 x 160 mm

Commit message: 이은혜
3/31
Parts:
- moved J2 164.8 mm to (-18.1, -174.7), turned to -90 degrees
- moved D40 163.8 mm to (-177.6, -86.2)
- moved Q39 163.8 mm to (-179.1, -92.4)
- moved R176 163.8 mm to (-178.1, -98.9)
- moved R190 163.8 mm to (-178.1, -97.2)
- moved R191 163.8 mm to (-178.1, -95.4)
- moved U79 163.8 mm to (-178.1, -104.3)
- moved J54 163.8 mm to (-176.6, -78.6)
- moved R187 163.7 mm to (-187.5, -95.4)
- moved U77 163.7 mm to (-187.4, -104.3)
- moved D38 163.7 mm to (-186.9, -86.3)
- moved J52 163.7 mm to (-185.9, -78.7)
- moved Q37 163.7 mm to (-188.4, -92.3)
- moved R174 163.7 mm to (-187.5, -99.0)
- moved R186 163.7 mm to (-187.5, -97.2)
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Routing:
- net /CLK: track 52.8 -> 8.39 mm
- net /S8: track 53.4 -> 13.7 mm
- net /S6: track 43.2 -> 3.69 mm
- net /S2: track 36.5 -> 1.90 mm
- net /S4: track 36.2 -> 2.85 mm
- net /DATA1_OUT: track 48.0 -> 14.7 mm
- net /LATCH: track 54.5 -> 21.2 mm
- net /S33: track 44.0 -> 15.2 mm
- net /S17: track 44.2 -> 17.1 mm
- net /S9: track 44.8 -> 18.0 mm
- net /S40: track 54.5 -> 28.9 mm
- net /S16: track 57.0 -> 31.7 mm
- net /S48: track 55.2 -> 30.4 mm
- net /S41: track 44.5 -> 22.7 mm
- net /S32: track 54.0 -> 32.9 mm
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Other:
- outline, holes or cut-outs redrawn
