File: NozzleControlBoard.kicad_sch (KiCad schematic)
At the start: 420 parts, among them IC2 MAX3094EESE+, IC3 MAX22245BAWA+, J1 24V_OUT, J10 SOL3, J101 SHIFT_DATA_TOSS, J102 8BIT_24V_IN, J103 SHIFT_DATA_TOSS, J104 8BIT_24V_OUT, J11 SOL4, J12 SOL5, J13 SOL6, J14 SOL7, J15 SOL8, J16 SOL9, J17 SOL10, J18 SOL11, J19 SOL12, J2 SHIFT_DATA_TOSS, J20 SOL13, J21 SOL14, J22 SOL15, J23 SOL16, J24 SOL17, J25 SOL18, J26 SOL19, J27 SOL20, J28 SOL21, J29 SOL22, J3 Conn_01x12_Male, J30 SOL23, J31 SOL24, J32 SOL25, J33 SOL26, J34 SOL27, J35 SOL28, J36 SOL29, J37 SOL30, J38 SOL31, J39 SOL32, J4 SHIFT_DATA_TOSS, J40 SOL33, J41 SOL34, J42 SOL35, J43 SOL36, J44 SOL37, J45 SOL38, J46 SOL39, J47 SOL40, J48 SOL41, J49 SOL42, J5 SHIFT_DATA_TOSS, J50 SOL43, J51 SOL44, J52 SOL45, J53 SOL46, J54 SOL47, J55 SOL48, J6 8BIT_24V_IN, J7 8BIT_24V_OUT, J8 SOL1, J9 SOL2, Q1 TPN22006NH,LQ, Q10 TPN22006NH,LQ, Q101 TPN22006NH,LQ, Q102 TPN22006NH,LQ, Q103 TPN22006NH,LQ, Q104 TPN22006NH,LQ, Q105 TPN22006NH,LQ, Q106 TPN22006NH,LQ, Q107 TPN22006NH,LQ, Q108 TPN22006NH,LQ, Q11 TPN22006NH,LQ, Q12 TPN22006NH,LQ, Q13 TPN22006NH,LQ, Q14 TPN22006NH,LQ, Q15 TPN22006NH,LQ, Q16 TPN22006NH,LQ, Q17 TPN22006NH,LQ, Q18 TPN22006NH,LQ, Q19 TPN22006NH,LQ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

Commit message: .
.
Parts:
- added C27, C30, C33, C38: 0.1uF, Capacitor_SMD:C_0603_1608Metric, symbol Device:C
- added C28, C31, C34, C39: 1uF, Capacitor_SMD:C_0603_1608Metric, symbol Device:C
- added C29, C32, C35, C43: 10uF, Capacitor_SMD:C_0603_1608Metric, symbol Device:C
- added D42, D43, D44, D45, D46, D47, D48, D49, D50, D51, D52, D53, D54, D55, D56, D57, D58, D59, D60, D61, D62, D63, D64, D65: DIODE, Diode_SMD:D_SMB, symbol pspice:DIODE
- added J56: 8BIT_24V_IN, 24V_PAD:24V_PAD, symbol Connector:Conn_01x02_Female
- added J57: SHIFT_DATA_TOSS, SHIFT_DATA_TOSS:SHIFT_DATA_TOSS, symbol Connector:Conn_01x08_Female
- added J58: SOL25, footprint:2PIN, symbol 2pin:22-04-1021
- added J59: SOL26, footprint:2PIN, symbol 2pin:22-04-1021
- added J60: SOL27, footprint:2PIN, symbol 2pin:22-04-1021
- added J61: SOL28, footprint:2PIN, symbol 2pin:22-04-1021
- added J62: SOL29, footprint:2PIN, symbol 2pin:22-04-1021
- added J63: SOL30, footprint:2PIN, symbol 2pin:22-04-1021
- added J64: SOL31, footprint:2PIN, symbol 2pin:22-04-1021
- added J65: SOL32, footprint:2PIN, symbol 2pin:22-04-1021
- added J66: SOL35, footprint:2PIN, symbol 2pin:22-04-1021
- added J67: SOL38, footprint:2PIN, symbol 2pin:22-04-1021
- added J68: SOL34, footprint:2PIN, symbol 2pin:22-04-1021
- added J69: SOL37, footprint:2PIN, symbol 2pin:22-04-1021
- added J70: SOL33, footprint:2PIN, symbol 2pin:22-04-1021
- added J71: SOL36, footprint:2PIN, symbol 2pin:22-04-1021
- added J72: SOL39, footprint:2PIN, symbol 2pin:22-04-1021
- added J73: SOL40, footprint:2PIN, symbol 2pin:22-04-1021
- added J74: SOL44, footprint:2PIN, symbol 2pin:22-04-1021
- added J75: SOL47, footprint:2PIN, symbol 2pin:22-04-1021
- added J76: SOL41, footprint:2PIN, symbol 2pin:22-04-1021
- added J77: SOL42, footprint:2PIN, symbol 2pin:22-04-1021
- added J78: SOL43, footprint:2PIN, symbol 2pin:22-04-1021
- added J79: SOL45, footprint:2PIN, symbol 2pin:22-04-1021
- added J80: SOL46, footprint:2PIN, symbol 2pin:22-04-1021
- added J81: SOL48, footprint:2PIN, symbol 2pin:22-04-1021
- added J82: SHIFT_DATA_TOSS, footprint:SHIFT_DATA_TOSS, symbol Connector:Conn_01x08_Female
- added J83: 8BIT_24V_OUT, 24V_PAD:24V_PAD, symbol Connector:Conn_01x02_Female
- added Q41, Q42, Q43, Q44, Q45, Q46, Q47, Q48, Q49, Q50, Q51, Q52, Q53, Q54, Q55, Q56, Q57, Q58, Q59, Q60, Q61, Q62, Q63, Q64: TPN22006NH,LQ, footprint:TPN22006NHLQ, symbol TPN22006NH:TPN22006NH,LQ
- added R100, R101, R102, R103, R104, R130, R163, R164, R165, R166, R167, R168, R169, R194, R195, R196, R197, R198, R199, R200, R201, R202, R211, R212, R213, R214, R215, R216, R217, R218, R219, R220, R221, R222, R223, R224, R225, R226, R89, R90, R91, R92, R93, R94, R95, R97, R98, R99: 22kΩ, Resistor_SMD:R_0603_1608Metric, symbol Device:R
- added R131, R132, R133, R134, R135, R136, R137, R162, R203, R204, R205, R206, R207, R208, R209, R210, R81, R82, R83, R84, R85, R86, R87, R88: 3.3kΩ, Resistor_SMD:R_0603_1608Metric, symbol Device:R
- added R80: 100Ω, Resistor_SMD:R_0603_1608Metric, symbol Device:R
- added U19: 74HC244, footprint:SOP65P640X110-20N, symbol 74xx:74HC244
- added U20, U21, U22, U23, U24, U25, U26, U35, U37, U38, U39, U40, U41, U42, U48, U49, U51, U52, U53, U54, U55, U65, U66, U67: TLP291, Package_SO:SOIC-4_4.55x2.6mm_P1.27mm, symbol Isolator:TLP291
- added U36, U50, U68: 74HCT595, Package_SO:SSOP-16_5.3x6.2mm_P0.65mm, symbol 74xx:74HCT595
- U4: footprint footprint:4PIN_ISP -> footprint:TPN22006NHLQ
Connections:
- net 24V2: now also J56.2 (Pin_2), J58.1, J59.1, J60.1, J61.1, J62.1, J63.1, J64.1, J65.1, J66.1, J67.1, J68.1, J69.1, J70.1, J71.1, J72.1, J73.1, J74.1, J75.1, J76.1, J77.1, J78.1, J79.1, J80.1, J81.1, J83.2 (Pin_2), U20.4, U21.4, U22.4, U23.4, U24.4, U25.4, U26.4, U35.4, U37.4, U38.4, U39.4, U40.4, U41.4, U42.4, U48.4, U49.4, U51.4, U52.4, U53.4, U54.4, U55.4, U65.4, U66.4, U67.4
- net 24V2_GND: now also D42.1 (K), D43.1 (K), D44.1 (K), D45.1 (K), D46.1 (K), D47.1 (K), D48.1 (K), D49.1 (K), D50.1 (K), D51.1 (K), D52.1 (K), D53.1 (K), D54.1 (K), D55.1 (K), D56.1 (K), D57.1 (K), D58.1 (K), D59.1 (K), D60.1 (K), D61.1 (K), D62.1 (K), D63.1 (K), D64.1 (K), D65.1 (K), J56.1 (Pin_1), J83.1 (Pin_1), Q41.1 (S_1), Q41.2 (S_2), Q41.3 (S_3), Q42.1 (S_1), Q42.2 (S_2), Q42.3 (S_3), Q43.1 (S_1), Q43.2 (S_2), Q43.3 (S_3), Q44.1 (S_1), Q44.2 (S_2), Q44.3 (S_3), Q45.1 (S_1), Q45.2 (S_2), Q45.3 (S_3), Q46.1 (S_1), Q46.2 (S_2), Q46.3 (S_3), Q47.1 (S_1), Q47.2 (S_2), Q47.3 (S_3), Q48.1 (S_1), Q48.2 (S_2), Q48.3 (S_3), Q49.1 (S_1), Q49.2 (S_2), Q49.3 (S_3), Q50.1 (S_1), Q50.2 (S_2), Q50.3 (S_3), Q51.1 (S_1), Q51.2 (S_2), Q51.3 (S_3), Q52.1 (S_1), Q52.2 (S_2), Q52.3 (S_3), Q53.1 (S_1), Q53.2 (S_2), Q53.3 (S_3), Q54.1 (S_1), Q54.2 (S_2), Q54.3 (S_3), Q55.1 (S_1), Q55.2 (S_2), Q55.3 (S_3), Q56.1 (S_1), Q56.2 (S_2), Q56.3 (S_3), Q57.1 (S_1), Q57.2 (S_2), Q57.3 (S_3), Q58.1 (S_1), Q58.2 (S_2), Q58.3 (S_3), Q59.1 (S_1), Q59.2 (S_2), Q59.3 (S_3), Q60.1 (S_1), Q60.2 (S_2), Q60.3 (S_3), Q61.1 (S_1), Q61.2 (S_2), Q61.3 (S_3), Q62.1 (S_1), Q62.2 (S_2), Q62.3 (S_3), Q63.1 (S_1), Q63.2 (S_2), Q63.3 (S_3), Q64.1 (S_1), Q64.2 (S_2), Q64.3 (S_3), R101.2, R103.2, R130.2, R164.2, R166.2, R168.2, R194.2, R196.2, R198.2, R200.2, R202.2, R212.2, R214.2, R216.2, R218.2, R220.2, R222.2, R224.2, R226.2, R90.2, R92.2, R94.2, R97.2, R99.2
- net 5V_3: now also J57.8 (Pin_8), J82.8 (Pin_8)
- net 5V_4: now also C27.2, C28.2, C29.1, C30.2, C31.2, C32.1, C33.2, C34.2, C35.1, C38.2, C39.2, C43.1, J57.5 (Pin_5), J82.5 (Pin_5), U19.20 (VCC), U20.1, U21.1, U22.1, U23.1, U24.1, U25.1, U26.1, U35.1, U36.10 (~{SRCLR}), U36.16 (VCC), U37.1, U38.1, U39.1, U40.1, U41.1, U42.1, U48.1, U49.1, U50.10 (~{SRCLR}), U50.16 (VCC), U51.1, U52.1, U53.1, U54.1, U55.1, U65.1, U66.1, U67.1, U68.10 (~{SRCLR}), U68.16 (VCC)
- net CLK2_IN: now also J57.4 (Pin_4), U19.2 (1A0)
- net CLK_3: now also J82.4 (Pin_4), U19.18 (1Y0), U36.11 (SRCLK), U50.11 (SRCLK), U68.11 (SRCLK)
- net DATA4_INPUT: now also U19.12 (1Y3), U36.14 (SER)
- net DATA4_INPUT_IN: now also J57.1 (Pin_1), U19.8 (1A3)
- net DATA4_OUT: now also U36.9 (QH'), U50.14 (SER)
- net DATA5_OUT: now also U50.9 (QH'), U68.14 (SER)
- net DATA6_OUT: now also J82.1 (Pin_1), U68.9 (QH')
- net ENABLE2_IN: now also J57.2 (Pin_2), U19.6 (1A2)
- net ENABLE_3: now also J82.2 (Pin_2), U19.14 (1Y2), U36.13 (~{OE}), U50.13 (~{OE}), U68.13 (~{OE})
- net GND_3: now also J57.7 (Pin_7), J82.7 (Pin_7)
- net GND_4: now also C27.1, C28.1, C29.2, C30.1, C31.1, C32.2, C33.1, C34.1, C35.2, C38.1, C39.1, C43.2, J57.6 (Pin_6), J82.6 (Pin_6), R80.1, U19.10 (GND), U36.8 (GND), U50.8 (GND), U68.8 (GND)
- net LATCH2_IN: now also J57.3 (Pin_3), U19.4 (1A1)
- net LATCH_3: now also J82.3 (Pin_3), U19.16 (1Y1), U36.12 (RCLK), U50.12 (RCLK), U68.12 (RCLK)
- net S25: now also R81.2, U36.15 (QA)
- net S26: now also R82.2, U36.1 (QB)
- net S27: now also R83.2, U36.2 (QC)
- net S28: now also R84.2, U36.3 (QD)
- net S29: now also R85.2, U36.4 (QE)
- net S30: now also R86.2, U36.5 (QF)
- net S31: now also R87.2, U36.6 (QG)
- net S32: now also R88.2, U36.7 (QH)
- net S33: now also R131.2, U50.15 (QA)
- net S34: now also R132.2, U50.1 (QB)
- net S35: now also R133.2, U50.2 (QC)
- net S36: now also R134.2, U50.3 (QD)
- net S37: now also R135.2, U50.4 (QE)
- net S38: now also R136.2, U50.5 (QF)
- net S39: now also R137.2, U50.6 (QG)
- net S40: now also R162.2, U50.7 (QH)
- net S41: now also R203.2, U68.15 (QA)
- net S42: now also R204.2, U68.1 (QB)
- net S43: now also R205.2, U68.2 (QC)
- net S44: now also R206.2, U68.3 (QD)
- net S45: now also R207.2, U68.4 (QE)
- net S46: now also R208.2, U68.5 (QF)
- net S47: now also R209.2, U68.6 (QG)
- net S48: now also R210.2, U68.7 (QH)
- net SOL25-: now also D42.2 (A), J58.2, Q41.5 (D_1), Q41.6 (D_2), Q41.7 (D_3), Q41.8 (D_4), Q41.9 (D_5)
- net SOL26-: now also D43.2 (A), J59.2, Q42.5 (D_1), Q42.6 (D_2), Q42.7 (D_3), Q42.8 (D_4), Q42.9 (D_5)
- net SOL27-: now also D44.2 (A), J60.2, Q43.5 (D_1), Q43.6 (D_2), Q43.7 (D_3), Q43.8 (D_4), Q43.9 (D_5)
- net SOL28-: now also D45.2 (A), J61.2, Q44.5 (D_1), Q44.6 (D_2), Q44.7 (D_3), Q44.8 (D_4), Q44.9 (D_5)
- net SOL29-: now also D46.2 (A), J62.2, Q45.5 (D_1), Q45.6 (D_2), Q45.7 (D_3), Q45.8 (D_4), Q45.9 (D_5)
- net SOL30-: now also D47.2 (A), J63.2, Q46.5 (D_1), Q46.6 (D_2), Q46.7 (D_3), Q46.8 (D_4), Q46.9 (D_5)
- net SOL31-: now also D48.2 (A), J64.2, Q47.5 (D_1), Q47.6 (D_2), Q47.7 (D_3), Q47.8 (D_4), Q47.9 (D_5)
- net SOL32-: now also D49.2 (A), J65.2, Q48.5 (D_1), Q48.6 (D_2), Q48.7 (D_3), Q48.8 (D_4), Q48.9 (D_5)
- net SOL33-: now also D50.2 (A), J70.2, Q49.5 (D_1), Q49.6 (D_2), Q49.7 (D_3), Q49.8 (D_4), Q49.9 (D_5)
- net SOL34-: now also D51.2 (A), J68.2, Q50.5 (D_1), Q50.6 (D_2), Q50.7 (D_3), Q50.8 (D_4), Q50.9 (D_5)
- net SOL35-: now also D52.2 (A), J66.2, Q51.5 (D_1), Q51.6 (D_2), Q51.7 (D_3), Q51.8 (D_4), Q51.9 (D_5)
- net SOL36-: now also D53.2 (A), J71.2, Q52.5 (D_1), Q52.6 (D_2), Q52.7 (D_3), Q52.8 (D_4), Q52.9 (D_5)
- net SOL37-: now also D54.2 (A), J69.2, Q53.5 (D_1), Q53.6 (D_2), Q53.7 (D_3), Q53.8 (D_4), Q53.9 (D_5)
- net SOL38-: now also D55.2 (A), J67.2, Q54.5 (D_1), Q54.6 (D_2), Q54.7 (D_3), Q54.8 (D_4), Q54.9 (D_5)
- net SOL39-: now also D56.2 (A), J72.2, Q55.5 (D_1), Q55.6 (D_2), Q55.7 (D_3), Q55.8 (D_4), Q55.9 (D_5)
- net SOL40-: now also D57.2 (A), J73.2, Q56.5 (D_1), Q56.6 (D_2), Q56.7 (D_3), Q56.8 (D_4), Q56.9 (D_5)
- net SOL41-: now also D58.2 (A), J76.2, Q57.5 (D_1), Q57.6 (D_2), Q57.7 (D_3), Q57.8 (D_4), Q57.9 (D_5)
- net SOL42-: now also D59.2 (A), J77.2, Q58.5 (D_1), Q58.6 (D_2), Q58.7 (D_3), Q58.8 (D_4), Q58.9 (D_5)
- net SOL43-: now also D60.2 (A), J78.2, Q59.5 (D_1), Q59.6 (D_2), Q59.7 (D_3), Q59.8 (D_4), Q59.9 (D_5)
- net SOL44-: now also D61.2 (A), J74.2, Q60.5 (D_1), Q60.6 (D_2), Q60.7 (D_3), Q60.8 (D_4), Q60.9 (D_5)
- net SOL45-: now also D62.2 (A), J79.2, Q61.5 (D_1), Q61.6 (D_2), Q61.7 (D_3), Q61.8 (D_4), Q61.9 (D_5)
- net SOL46-: now also D63.2 (A), J80.2, Q62.5 (D_1), Q62.6 (D_2), Q62.7 (D_3), Q62.8 (D_4), Q62.9 (D_5)
- net SOL47-: now also D64.2 (A), J75.2, Q63.5 (D_1), Q63.6 (D_2), Q63.7 (D_3), Q63.8 (D_4), Q63.9 (D_5)
- net SOL48-: now also D65.2 (A), J81.2, Q64.5 (D_1), Q64.6 (D_2), Q64.7 (D_3), Q64.8 (D_4), Q64.9 (D_5)
- new net: R85.1, U24.2
- new net: R98.2, U24.3
- new net: R208.1, U65.2
- new net: R221.2, U65.3
- new net: Q61.4 (G), R219.1, R220.1
- new net: Q53.4 (G), R195.1, R196.1
- new net: R203.1, U51.2
- new net: R211.2, U51.3
- new net: R135.1, U41.2
- new net: R195.2, U41.3
- new net: Q44.4 (G), R95.1, R97.1
- new net: R95.2, U23.3
- new net: Q62.4 (G), R221.1, R222.1
- new net: R131.1, U37.2
- new net: Q51.4 (G), R167.1, R168.1
- new net: R167.2, U39.3
- new net: Q57.4 (G), R211.1, R212.1
- new net: Q60.4 (G), R217.1, R218.1
- new net: R88.1, U35.2
- new net: R104.2, U35.3
- new net: R132.1, U38.2
- new net: R209.1, U66.2
- new net: Q45.4 (G), R98.1, R99.1
- new net: R84.1, U23.2
- new net: R207.1, U55.2
- new net: R204.1, U52.2
- new net: R86.1, U25.2
- new net: R100.2, U25.3
- new net: Q54.4 (G), R197.1, R198.1
- new net: R197.2, U42.3
- new net: Q41.4 (G), R89.1, R90.1
- new net: R89.2, U20.3
- new net: Q43.4 (G), R93.1, R94.1
- new net: R93.2, U22.3
- new net: Q47.4 (G), R102.1, R103.1
- new net: R134.1, U40.2
- new net: R169.2, U40.3
- new net: R83.1, U22.2
- new net: R82.1, U21.2
- new net: R91.2, U21.3
- new net: R219.2, U55.3
- new net: Q50.4 (G), R165.1, R166.1
- new net: R165.2, U38.3
- new net: Q58.4 (G), R213.1, R214.1
- new net: R213.2, U52.3
- new net: R205.1, U53.2
- new net: Q49.4 (G), R163.1, R164.1
- new net: Q59.4 (G), R215.1, R216.1
- new net: R223.2, U66.3
- new net: Q63.4 (G), R223.1, R224.1
- new net: Q64.4 (G), R225.1, R226.1
- new net: R225.2, U67.3
- new net: R206.1, U54.2
- new net: R217.2, U54.3
- new net: R80.2, U19.1 (1OE), U19.19 (2OE)
- new net: Q48.4 (G), R104.1, R130.1
- new net: R163.2, U37.3
- new net: Q42.4 (G), R91.1, R92.1
- new net: R162.1, U49.2
- new net: R210.1, U67.2
- new net: R137.1, U48.2
- new net: R199.2, U48.3
- new net: R215.2, U53.3
- new net: Q56.4 (G), R201.1, R202.1
- new net: Q46.4 (G), R100.1, R101.1
- new net: R87.1, U26.2
- new net: R102.2, U26.3
- new net: R201.2, U49.3
- new net: Q52.4 (G), R169.1, R194.1
- new net: Q55.4 (G), R199.1, R200.1
- new net: R133.1, U39.2
- new net: R81.1, U20.2
- new net: R136.1, U42.2

Commit message: .
.
Parts:
- removed J1: 24V_OUT, footprint:24V_PAD, symbol Connector:Conn_01x02_Female
- removed J101, J4, J5, J57: SHIFT_DATA_TOSS, SHIFT_DATA_TOSS:SHIFT_DATA_TOSS, symbol Connector:Conn_01x08_Female
- removed J102, J56, J6: 8BIT_24V_IN, 24V_PAD:24V_PAD, symbol Connector:Conn_01x02_Female
- removed J2, J82: SHIFT_DATA_TOSS, footprint:SHIFT_DATA_TOSS, symbol Connector:Conn_01x08_Female
- removed J7, J83: 8BIT_24V_OUT, 24V_PAD:24V_PAD, symbol Connector:Conn_01x02_Female
- removed U101: 74HC244, footprint:SOP65P640X110-20N, symbol 74xx:74HC244
- removed U20, U37, U51, U52: TLP291, Package_SO:SOIC-4_4.55x2.6mm_P1.27mm, symbol Isolator:TLP291
- removed U36, U50: 74HCT595, Package_SO:SSOP-16_5.3x6.2mm_P0.65mm, symbol 74xx:74HCT595
- added C100, C104, C47, C54, C61, C70, C73, C76, C79, C82, C85, C88, C91, C94, C97: 0.1uF, Capacitor_SMD:C_0603_1608Metric, symbol Device:C
- added C101, C50, C56, C68, C71, C74, C77, C80, C83, C86, C89, C92, C95, C98: 1uF, Capacitor_SMD:C_0603_1608Metric, symbol Device:C
- added C102, C103, C52, C59, C69, C72, C75, C78, C81, C84, C87, C90, C93, C96, C99: 10uF, Capacitor_SMD:C_0603_1608Metric, symbol Device:C
- added D100, D109, D110, D111, D112, D113, D114, D115, D116, D117, D118, D119, D120, D121, D122, D123, D124, D125, D126, D127, D128, D129, D130, D131, D132, D133, D134, D135, D136, D137, D138, D139, D140, D141, D66, D67, D68, D69, D70, D71, D72, D73, D74, D75, D76, D77, D78, D79, D80, D81, D82, D83, D84, D85, D86, D87, D88, D89, D90, D91, D92, D93, D94, D95, D96, D97, D98, D99: DIODE, Diode_SMD:D_SMB, symbol pspice:DIODE
- added J1, J106, J122: SOL35, footprint:2PIN, symbol 2pin:22-04-1021
- added J100: SOL29, footprint:2PIN, symbol 2pin:22-04-1021
- added J101: SOL30, footprint:2PIN, symbol 2pin:22-04-1021
- added J102: SOL31, footprint:2PIN, symbol 2pin:22-04-1021
- added J105: SOL32, footprint:2PIN, symbol 2pin:22-04-1021
- added J107, J123, J2: SOL38, footprint:2PIN, symbol 2pin:22-04-1021
- added J108, J124, J4: SOL34, footprint:2PIN, symbol 2pin:22-04-1021
- added J109, J125, J5: SOL37, footprint:2PIN, symbol 2pin:22-04-1021
- added J110, J126, J6: SOL33, footprint:2PIN, symbol 2pin:22-04-1021
- added J111, J127, J7: SOL36, footprint:2PIN, symbol 2pin:22-04-1021
- added J112, J128, J56: SOL39, footprint:2PIN, symbol 2pin:22-04-1021
- added J113, J129, J57: SOL40, footprint:2PIN, symbol 2pin:22-04-1021
- added J114, J130, J138: SOL44, footprint:2PIN, symbol 2pin:22-04-1021
- added J115, J131: SOL47, footprint:2PIN, symbol 2pin:22-04-1021
- added J116, J132, J139: SOL41, footprint:2PIN, symbol 2pin:22-04-1021
- added J117, J133, J140: SOL42, footprint:2PIN, symbol 2pin:22-04-1021
- added J118, J134, J141: SOL43, footprint:2PIN, symbol 2pin:22-04-1021
- added J119, J135, J142: SOL45, footprint:2PIN, symbol 2pin:22-04-1021
- added J120, J136, J143: SOL46, footprint:2PIN, symbol 2pin:22-04-1021
- added J121, J137: SOL48, footprint:2PIN, symbol 2pin:22-04-1021
- added J144: SHIFT_DATA_TOSS, footprint:SHIFT_DATA_TOSS, symbol Connector:Conn_01x08_Female
- added J145: 8BIT_24V_OUT, 24V_PAD:24V_PAD, symbol Connector:Conn_01x02_Female
- added J82: SOL9, footprint:2PIN, symbol 2pin:22-04-1021
- added J83: SOL10, footprint:2PIN, symbol 2pin:22-04-1021
- added J84: SOL11, footprint:2PIN, symbol 2pin:22-04-1021
- added J85: SOL12, footprint:2PIN, symbol 2pin:22-04-1021
- added J86: SOL13, footprint:2PIN, symbol 2pin:22-04-1021
- added J87: SOL16, footprint:2PIN, symbol 2pin:22-04-1021
- added J88: SOL17, footprint:2PIN, symbol 2pin:22-04-1021
- added J89: SOL18, footprint:2PIN, symbol 2pin:22-04-1021
- added J90: SOL19, footprint:2PIN, symbol 2pin:22-04-1021
- added J91: SOL20, footprint:2PIN, symbol 2pin:22-04-1021
- added J92: SOL21, footprint:2PIN, symbol 2pin:22-04-1021
- added J93: SOL22, footprint:2PIN, symbol 2pin:22-04-1021
- added J94: SOL23, footprint:2PIN, symbol 2pin:22-04-1021
- added J95: SOL24, footprint:2PIN, symbol 2pin:22-04-1021
- added J96: SOL25, footprint:2PIN, symbol 2pin:22-04-1021
- added J97: SOL26, footprint:2PIN, symbol 2pin:22-04-1021
- added J98: SOL27, footprint:2PIN, symbol 2pin:22-04-1021
- added J99: SOL28, footprint:2PIN, symbol 2pin:22-04-1021
- added PS2: R05CTE05S-R, footprint:SOIC127P1030X265-16N, symbol R05CTE05S:R05CTE05S-R
- added Q100, Q109, Q110, Q111, Q112, Q113, Q114, Q115, Q116, Q117, Q118, Q119, Q120, Q121, Q122, Q123, Q124, Q125, Q126, Q127, Q128, Q129, Q130, Q131, Q132, Q133, Q134, Q135, Q136, Q137, Q138, Q139, Q140, Q65, Q67, Q68, Q69, Q70, Q71, Q72, Q73, Q74, Q75, Q76, Q77, Q78, Q79, Q80, Q81, Q82, Q83, Q84, Q85, Q86, Q87, Q88, Q89, Q90, Q91, Q92, Q93, Q94, Q95, Q96, Q97, Q98, Q99: TPN22006NH,LQ, footprint:TPN22006NHLQ, symbol TPN22006NH:TPN22006NH,LQ
- added Q66: TPN22006NH,LQ, TPN22006NH:TPN22006NHLQ, symbol TPN22006NH:TPN22006NH,LQ
- added R227, R228, R229, R246, R247, R248, R249, R250, R251, R252, R253, R271, R272, R273, R274, R275, R276, R277, R278, R295, R296, R297, R298, R299, R300, R301, R302, R320, R321, R322, R323, R324, R325, R326, R327, R344, R345, R346, R347, R348, R349, R350, R351, R369, R370, R371, R372, R373, R374, R375, R376, R393, R394, R395, R396, R397, R398, R399, R400, R417, R418, R419, R420, R421, R422: 3.3kΩ, Resistor_SMD:R_0603_1608Metric, symbol Device:R
- added R230, R231, R232, R233, R234, R235, R236, R237, R238, R239, R240, R241, R242, R243, R244, R245, R254, R255, R256, R257, R258, R259, R260, R261, R262, R263, R264, R265, R266, R267, R268, R269, R279, R280, R281, R282, R283, R284, R285, R286, R287, R288, R289, R290, R291, R292, R293, R294, R303, R304, R305, R306, R307, R308, R309, R310, R311, R312, R313, R314, R315, R316, R317, R318, R328, R329, R330, R331, R332, R333, R334, R335, R336, R337, R338, R339, R340, R341, R342, R343, R352, R353, R354, R355, R356, R357, R358, R359, R360, R361, R362, R363, R364, R365, R366, R367, R377, R378, R379, R380, R381, R382, R383, R384, R385, R386, R387, R388, R389, R390, R391, R392, R401, R402, R403, R404, R405, R406, R407, R408, R409, R410, R411, R412, R413, R414, R415, R416, R423, R424, R425, R426, R427, R428, R429, R430, R431, R432, R433, R434: 22kΩ, Resistor_SMD:R_0603_1608Metric, symbol Device:R
- added R270, R319, R368, R435: 100Ω, Resistor_SMD:R_0603_1608Metric, symbol Device:R
- added U100, U101, U111, U112, U113, U115, U116, U117, U118, U119, U120, U121, U122, U125, U126, U127, U128, U129, U130, U131, U132, U134, U135, U136, U137, U138, U139, U140, U141, U144, U145, U146, U147, U148, U149, U150, U151, U153, U154, U155, U156, U157, U158, U159, U160, U162, U163, U164, U165, U166, U167, U36, U50, U69, U70, U71, U72, U82, U83, U84, U85, U87, U88, U89, U90, U91, U92, U93, U94, U97, U98, U99: TLP291, Package_SO:SOIC-4_4.55x2.6mm_P1.27mm, symbol Isolator:TLP291
- added U114, U123, U133, U142, U152, U161, U168, U37, U51, U86, U95: 74HCT595, Package_SO:SSOP-16_5.3x6.2mm_P0.65mm, symbol 74xx:74HCT595
- added U124, U143, U169, U20, U52, U96: 74HC244, footprint:SOP65P640X110-20N, symbol 74xx:74HC244
- J58: value SOL25 -> SOL44
- J59: value SOL26 -> SOL47
- J60: value SOL27 -> SOL41
- J61: value SOL28 -> SOL42
- J62: value SOL29 -> SOL43
- J63: value SOL30 -> SOL45
- J64: value SOL31 -> SOL46
- J65: value SOL32 -> SOL48
- J66: value SOL35 -> SOL44
- J67: value SOL38 -> SOL41
- J68: value SOL34 -> SOL42
- J69: value SOL37 -> SOL43
- J70: value SOL33 -> SOL45
- J71: value SOL36 -> SOL46
- J72: value SOL39 -> SOL5
- J73: value SOL40 -> SOL6
- J74: value SOL44 -> SOL7
- J75: value SOL47 -> SOL8
- J76: value SOL41 -> SOL71
- J77: value SOL42 -> SOL72
- J78: value SOL43 -> SOL3
- J79: value SOL45 -> SOL4
- J80: value SOL46 -> SOL15
- J81: value SOL48 -> SOL14
- R105: value 100Ω -> 22kΩ
- R203, R81: value 3.3kΩ -> 100Ω
- R210: value 3.3kΩ -> 22kΩ
- R222, R223, R224, R225, R226, R89: value 22kΩ -> 3.3kΩ
Connections:
- net CLK2_IN is gone; now on net CLK_2: U19.2 (1A0)
- net DATA3_INPUT is gone; now on net DATA3: U47.14 (SER), U5.12 (1Y3)
- net DATA3_INPUT_IN is gone; now on net DATA2: U5.8 (1A3)
- net DATA3_OUT is gone; now on net DATA4: U47.9 (QH')
- net ENABLE2_IN is gone; now on net ENABLE_2: U19.6 (1A2)
- net LATCH2_IN is gone; now on net LATCH_2: U19.4 (1A1)
- net 24V2: now also J1.1, J100.1, J101.1, J102.1, J105.1, J106.1, J107.1, J108.1, J109.1, J110.1, J111.1, J112.1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
- net 24V2_GND: now also R100.2, R102.2, R104.2, R211.2, R213.2, R215.2, R217.2, R219.2, R221.2, R91.2, R93.2, R95.2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; no longer R101.2, R103.2, R212.2, R214.2, R216.2, R218.2, R220.2, R222.2, R224.2, R226.2, R90.2, R92.2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
- net 5V_3: now also J144.8 (Pin_8), PS2.3 (+VIN_1), PS2.4 (+VIN_2)
- net 5V_4: now also C100.2, C101.2, C102.1, C47.2, C50.2, C52.1, C54.2, C56.2, C59.1, C61.2, C68.2, C69.1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
- net CLK_2: now also U102.11 (SRCLK), U114.11 (SRCLK), U123.11 (SRCLK), U124.2 (1A0)
- net CLK_3: now also U124.18 (1Y0), U133.11 (SRCLK), U142.11 (SRCLK), U143.2 (1A0), U20.2 (1A0); no longer J103.4 (Pin_4), U102.11 (SRCLK), U68.11 (SRCLK)
- net DATA3: now also U114.14 (SER)
- net DATA4: now also U102.14 (SER), U114.9 (QH'), U123.14 (SER)
- net ENABLE_2: now also U102.13 (~{OE}), U114.13 (~{OE}), U123.13 (~{OE}), U124.6 (1A2)
- net ENABLE_3: now also U124.14 (1Y2), U133.13 (~{OE}), U142.13 (~{OE}), U143.6 (1A2), U20.6 (1A2); no longer J103.2 (Pin_2), U102.13 (~{OE}), U68.13 (~{OE})
- net GND_3: now also J144.6 (Pin_6), J144.7 (Pin_7), PS2.1 (-VIN_1), PS2.2 (-VIN_2), PS2.5 (SGNDIN_1), PS2.6 (SGNDIN_2), PS2.7 (SGNDIN_3), PS2.8 (SGNDIN_4)
- net GND_4: now also R203.1, R81.1, C100.1, C101.1, C102.2, C47.1, C50.1, C52.2, C54.1, C56.1, C59.2, C61.1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; no longer R105.1
- net LATCH_2: now also U102.12 (RCLK), U114.12 (RCLK), U123.12 (RCLK), U124.4 (1A1)
- net LATCH_3: now also U124.16 (1Y1), U133.12 (RCLK), U142.12 (RCLK), U143.4 (1A1), U20.4 (1A1); no longer J103.3 (Pin_3), U102.12 (RCLK), U68.12 (RCLK)
- net S1: now also R222.2, U86.15 (QA)
- net S10: now also R247.2, U95.1 (QB)
- net S11: now also R248.2, U95.2 (QC)
- net S12: now also R249.2, U95.3 (QD)
- net S13: now also R250.2, U95.4 (QE)
- net S14: now also R251.2, U95.5 (QF)
- net S15: now also R252.2, U95.6 (QG)
- net S16: now also R253.2, U95.7 (QH)
- net S17: now also R271.2, U114.15 (QA)
- net S18: now also R272.2, U114.1 (QB)
- net S19: now also R273.2, U114.2 (QC)
- net S2: now also R223.2, U86.1 (QB)
- net S20: now also R274.2, U114.3 (QD)
- net S21: now also R275.2, U114.4 (QE)
- net S22: now also R276.2, U114.5 (QF)
- net S23: now also R277.2, U114.6 (QG)
- net S24: now also R278.2, U114.7 (QH)
- net S25: now also R295.2, U123.15 (QA); no longer R81.2
- net S26: now also R296.2, U123.1 (QB); no longer R82.2
- net S27: now also R297.2, U123.2 (QC); no longer R83.2
- net S28: now also R298.2, U123.3 (QD); no longer R84.2
- net DATA1_OUT renamed DATA1
- net DATA2_OUT renamed DATA2
- net DATA4_INPUT renamed DATA6
- net DATA4_INPUT_IN renamed DATA5
- removed net DATA4_OUT: U102.9 (QH'), U64.14 (SER)
- net DATA5_OUT renamed DATA7
- removed net DATA6_OUT: J103.1 (Pin_1), U68.9 (QH'), U81.9 (QH')
- net DATA_IN renamed DATA0
- new net: Q97.4 (G), R332.1, R333.1
- new net: R332.2, U127.3
- new net: R301.1, U121.2
- new net: R397.1, U157.2
- new net: R409.2, U157.3
- new net: R421.1, U166.2
- new net: R431.2, U166.3
- new net: R203.2, U52.1 (1OE), U52.19 (2OE)
- new net: Q95.4 (G), R328.1, R329.1
- new net: R328.2, U125.3
- new net: Q137.4 (G), R427.1, R428.1
- new net: R275.1, U101.2
- new net: Q76.4 (G), R264.1, R265.1
- new net: R264.2, U92.3
- new net: R393.1, U153.2
- new net: R323.1, U128.2
- new net: R334.2, U128.3
- new net: R250.1, U91.2
- new net: R262.2, U91.3
- new net: Q86.4 (G), R293.1, R294.1
- new net: R293.2, U113.3
- new net: R325.1, U130.2
- new net: R271.1, U97.2
- new net: Q85.4 (G), R291.1, R292.1
- new net: Q122.4 (G), R383.1, R384.1
- new net: Q115.4 (G), R360.1, R361.1
- new net: R376.1, U151.2
- new net: R391.2, U151.3
- new net: R435.2, U169.1 (1OE), U169.19 (2OE)
- new net: R251.1, U92.2
- new net: R326.1, U131.2
- new net: Q110.4 (G), R342.1, R343.1
- new net: Q98.4 (G), R334.1, R335.1
- new net: R295.1, U115.2
- new net: Q90.4 (G), R309.1, R310.1
- new net: R277.1, U112.2
- new net: Q127.4 (G), R401.1, R402.1
- new net: R401.2, U153.3
- new net: Q129.4 (G), R405.1, R406.1
- new net: R315.2, U121.3
- new net: R398.1, U158.2
- new net: Q65.4 (G), R234.1, R235.1
- new net: R227.1, U83.2
- new net: R287.2, U101.3
- new net: Q84.4 (G), R289.1, R290.1
- new net: Q66.4 (G), R236.1, R237.1
- new net: R319.2, U124.1 (1OE), U124.19 (2OE)
- new net: Q81.4 (G), R283.1, R284.1
- new net: R283.2, U99.3
- new net: Q83.4 (G), R287.1, R288.1
- new net: Q88.4 (G), R305.1, R306.1
- new net: Q92.4 (G), R313.1, R314.1
- new net: R313.2, U120.3
- new net: R422.1, U167.2
- new net: R433.2, U167.3
- new net: Q134.4 (G), R415.1, R416.1
- new net: R415.2, U160.3
- new net: R289.2, U111.3
- new net: R253.1, U94.2
- new net: Q70.4 (G), R244.1, R245.1
- new net: R225.1, U72.2
- new net: R372.1, U147.2
- new net: R383.2, U147.3
- new net: R229.1, U85.2
- new net: R244.2, U85.3
- new net: Q78.4 (G), R268.1, R269.1
- new net: Q138.4 (G), R429.1, R430.1
- new net: R429.2, U165.3
- new net: R246.1, U87.2
- new net: R254.2, U87.3
- new net: Q75.4 (G), R262.1, R263.1
- new net: R137.1, U49.2
- new net: R350.1, U140.2
- new net: R364.2, U140.3
- new net: Q131.4 (G), R409.1, R410.1
- new net: R349.1, U139.2
- new net: R362.2, U139.3
- new net: Q109.4 (G), R340.1, R341.1
- new net: R340.2, U131.3
- new net: Q136.4 (G), R425.1, R426.1
- new net: R425.2, U163.3
- new net: R273.1, U99.2
- new net: R418.1, U163.2
- new net: Q112.4 (G), R354.1, R355.1
- new net: Q125.4 (G), R389.1, R390.1
- new net: R389.2, U150.3
- new net: Q68.4 (G), R240.1, R241.1
- new net: R371.1, U146.2
- new net: Q118.4 (G), R366.1, R367.1
- new net: Q139.4 (G), R431.1, R432.1
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Other:
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
Commit message: 이은혜
3/31
Parts:
- J1: value SOL35 -> SOL51
- J100: value SOL29 -> SOL99
- J101: value SOL30 -> SOL100
- J102: value SOL31 -> SOL101
- J105: value SOL32 -> SOL102
- J106: value SOL35 -> SOL105
- J107: value SOL38 -> SOL108
- J108: value SOL34 -> SOL104
- J109: value SOL37 -> SOL107
- J110: value SOL33 -> SOL103
- J111: value SOL36 -> SOL106
- J112: value SOL39 -> SOL109
- J113: value SOL40 -> SOL110
- J122: value SOL35 -> SOL121
- J123: value SOL38 -> SOL124
- J124: value SOL34 -> SOL120
- J125: value SOL37 -> SOL123
- J126: value SOL33 -> SOL119
- J127: value SOL36 -> SOL122
- J128: value SOL39 -> SOL125
- J129: value SOL40 -> SOL126
- J130: value SOL44 -> SOL130
- J131: value SOL47 -> SOL133
- J132: value SOL41 -> SOL127
- J133: value SOL42 -> SOL128
- J134: value SOL43 -> SOL129
- J135: value SOL45 -> SOL131
- J136: value SOL46 -> SOL132
- J137: value SOL48 -> SOL134
- J138: value SOL44 -> SOL138
- J139: value SOL41 -> SOL135
- J140: value SOL42 -> SOL136
- J141: value SOL43 -> SOL137
- J142: value SOL45 -> SOL139
- J143: value SOL46 -> SOL140
- J2: value SOL38 -> SOL54
- J4: value SOL34 -> SOL50
- J5: value SOL37 -> SOL53
- J56: value SOL39 -> SOL55
- J57: value SOL40 -> SOL56
- J58: value SOL44 -> SOL60
- J59: value SOL47 -> SOL63
- J6: value SOL33 -> SOL49
- J60: value SOL41 -> SOL57
- J61: value SOL42 -> SOL58
- J62: value SOL43 -> SOL59
- J63: value SOL45 -> SOL61
- J64: value SOL46 -> SOL62
- J65: value SOL48 -> SOL64
- J66: value SOL44 -> SOL68
- J67: value SOL41 -> SOL65
- J68: value SOL42 -> SOL66
- J69: value SOL43 -> SOL67
- J7: value SOL36 -> SOL52
- J70: value SOL45 -> SOL69
- J71: value SOL46 -> SOL70
- J72: value SOL5 -> SOL75
- J73: value SOL6 -> SOL76
- J74: value SOL7 -> SOL77
- J75: value SOL8 -> SOL78
- J78: value SOL3 -> SOL73
- J79: value SOL4 -> SOL74
- J80: value SOL15 -> SOL85
- J81: value SOL14 -> SOL84
- J82: value SOL9 -> SOL79
- J83: value SOL10 -> SOL80
- J84: value SOL11 -> SOL81
- J85: value SOL12 -> SOL82
- J86: value SOL13 -> SOL83
- J87: value SOL16 -> SOL86
- J88: value SOL17 -> SOL87
- J89: value SOL18 -> SOL88
- J90: value SOL19 -> SOL89
- J91: value SOL20 -> SOL90
- J92: value SOL21 -> SOL91
- J93: value SOL22 -> SOL92
- J94: value SOL23 -> SOL93
- J95: value SOL24 -> SOL94
- J96: value SOL25 -> SOL95
- J97: value SOL26 -> SOL96
- J98: value SOL27 -> SOL97
- J99: value SOL28 -> SOL98
Connections:
- net CLK_2: no longer U114.11 (SRCLK), U123.11 (SRCLK), U124.2 (1A0)
- net CLK_3: no longer U124.18 (1Y0), U133.11 (SRCLK), U142.11 (SRCLK), U143.2 (1A0)
- net CLK_4: no longer U143.18 (1Y0), U152.11 (SRCLK), U161.11 (SRCLK), U168.11 (SRCLK), U169.2 (1A0)
- net CLK_5: no longer U169.18 (1Y0)
- net CLK_7: now also U114.11 (SRCLK), U123.11 (SRCLK), U124.2 (1A0)
- net DATA10: now also U37.9 (QH'); no longer U152.14 (SER), U37.14 (SER)
- net DATA11: now also U51.9 (QH'), U68.14 (SER); no longer U152.9 (QH'), U37.9 (QH')
- net DATA12: now also U52.8 (1A3), U68.9 (QH')
- net DATA13: now also J144.1 (Pin_1), U52.12 (1Y3), U86.14 (SER); no longer U161.9 (QH'), U168.14 (SER), U51.9 (QH'), U68.14 (SER)
- net DATA14: now also U86.9 (QH'), U95.14 (SER); no longer U168.9 (QH'), U169.8 (1A3), U52.8 (1A3), U68.9 (QH')
- net DATA15: now also U95.9 (QH'), U96.8 (1A3); no longer U169.12 (1Y3), U52.12 (1Y3)
- net DATA16: now also U114.14 (SER), U96.12 (1Y3); no longer J144.1 (Pin_1), U86.14 (SER)
- net DATA17: now also U114.9 (QH'), U123.14 (SER); no longer U86.9 (QH'), U95.14 (SER)
- net DATA18: now also U123.9 (QH'), U124.8 (1A3); no longer U95.9 (QH'), U96.8 (1A3)
- net DATA19: now also U124.12 (1Y3), U133.14 (SER); no longer U96.12 (1Y3)
- net DATA3: no longer U114.14 (SER)
- net DATA4: no longer U114.9 (QH'), U123.14 (SER)
- net DATA5: no longer U123.9 (QH'), U124.8 (1A3)
- net DATA6: no longer U124.12 (1Y3), U133.14 (SER)
- net DATA7: no longer U133.9 (QH'), U142.14 (SER)
- net DATA8: no longer U142.9 (QH'), U143.8 (1A3)
- net DATA9: now also U37.14 (SER); no longer U143.12 (1Y3)
- net ENABLE_2: no longer U114.13 (~{OE}), U123.13 (~{OE}), U124.6 (1A2)
- net ENABLE_3: no longer U124.14 (1Y2), U133.13 (~{OE}), U142.13 (~{OE}), U143.6 (1A2)
- net ENABLE_4: no longer U143.14 (1Y2), U152.13 (~{OE}), U161.13 (~{OE}), U168.13 (~{OE}), U169.6 (1A2)
- net ENABLE_5: no longer U169.14 (1Y2)
- net ENABLE_7: now also U114.13 (~{OE}), U123.13 (~{OE}), U124.6 (1A2)
- net LATCH_2: no longer U114.12 (RCLK), U123.12 (RCLK), U124.4 (1A1)
- net LATCH_3: no longer U124.16 (1Y1), U133.12 (RCLK), U142.12 (RCLK), U143.4 (1A1)
- net LATCH_4: no longer U143.16 (1Y1), U152.12 (RCLK), U161.12 (RCLK), U168.12 (RCLK), U169.4 (1A1)
- net LATCH_5: no longer U169.16 (1Y1)
- net LATCH_7: now also U114.12 (RCLK), U123.12 (RCLK), U124.4 (1A1)
- net S1: no longer R222.2
- net S10: no longer R247.2
- net S11: no longer R248.2
- net S12: no longer R249.2
- net S13: no longer R250.2
- net S14: no longer R251.2
- net S15: no longer R252.2
- net S16: no longer R253.2
- net S17: no longer R271.2
- net S18: no longer R272.2
- net S19: no longer R273.2
- net S2: no longer R223.2
- net S20: no longer R274.2
- net S21: no longer R275.2
- net S22: no longer R276.2
- net S23: no longer R277.2
- net S24: no longer R278.2
- net S25: no longer R295.2
- net S26: no longer R296.2
- net S27: no longer R297.2
- net S28: no longer R298.2
- net S29: no longer R299.2
- net S3: no longer R224.2
- net S30: no longer R300.2
- net S31: no longer R301.2
- net S32: no longer R302.2
- net S33: no longer R320.2, R369.2, R82.2
- net S34: no longer R321.2, R370.2, R83.2
- net S35: no longer R322.2, R371.2, R84.2
- net S36: no longer R323.2, R372.2, R85.2
- net S37: no longer R324.2, R373.2, R86.2
- net S38: no longer R325.2, R374.2, R87.2
- net S39: no longer R326.2, R375.2, R88.2
- net S4: no longer R225.2
- net S40: no longer R327.2, R376.2, R89.2
- net S41: no longer R131.2, R204.2, R344.2, R393.2, R417.2
- net S42: no longer R132.2, R205.2, R345.2, R394.2, R418.2
- net S43: no longer R133.2, R206.2, R346.2, R395.2, R419.2
- new net 78: R229.2
- new net CLK_10: U169.18 (1Y0)
- new net CLK_8: U124.18 (1Y0), U133.11 (SRCLK), U142.11 (SRCLK), U143.2 (1A0)
- new net CLK_9: U143.18 (1Y0), U152.11 (SRCLK), U161.11 (SRCLK), U168.11 (SRCLK), U169.2 (1A0)
- new net DATA20: U133.9 (QH'), U142.14 (SER)
- new net DATA21: U142.9 (QH'), U143.8 (1A3)
- new net DATA22: U143.12 (1Y3), U152.14 (SER)
- new net DATA23: U152.9 (QH')
- new net DATA24: U161.9 (QH'), U168.14 (SER)
- new net DATA25: U168.9 (QH'), U169.8 (1A3)
- new net DATA26: U169.12 (1Y3)
- new net ENABLE_10: U169.14 (1Y2)
- new net ENABLE_8: U124.14 (1Y2), U133.13 (~{OE}), U142.13 (~{OE}), U143.6 (1A2)
- new net ENABLE_9: U143.14 (1Y2), U152.13 (~{OE}), U161.13 (~{OE}), U168.13 (~{OE}), U169.6 (1A2)
- new net LATCH_10: U169.16 (1Y1)
- new net LATCH_8: U124.16 (1Y1), U133.12 (RCLK), U142.12 (RCLK), U143.4 (1A1)
- new net LATCH_9: U143.16 (1Y1), U152.12 (RCLK), U161.12 (RCLK), U168.12 (RCLK), U169.4 (1A1)
- new net S100: R300.2
- new net S101: R301.2
- new net S102: R302.2
- new net S103: R320.2
- new net S104: R321.2
- new net S105: R322.2
- new net S106: R323.2
- new net S107: R324.2
- new net S108: R325.2
- new net S109: R326.2
- new net S110: R327.2
- new net S111: R344.2
- new net S112: R345.2
- new net S113: R346.2
- new net S114: R347.2
- new net S115: R348.2
- new net S116: R349.2
- new net S117: R350.2
- new net S118: R351.2
- new net S119: R369.2
- new net S120: R370.2
- new net S121: R371.2
- new net S122: R372.2
- new net S123: R373.2
- new net S124: R374.2
- new net S125: R375.2
- new net S126: R376.2
- new net S127: R393.2
- new net S128: R394.2
- new net S129: R395.2
- new net S130: R396.2
- new net S131: R397.2
- new net S132: R398.2
- new net S133: R399.2
- new net S134: R400.2
- new net S135: R417.2
- new net S136: R418.2
- new net S137: R419.2
- new net S138: R420.2
- new net S139: R421.2
- new net S140: R422.2
- new net S49: R82.2
- new net S50: R83.2
- new net S51: R84.2
- new net S52: R85.2
- new net S53: R86.2
- new net S54: R87.2
- new net S55: R88.2
- new net S56: R89.2
- new net S57: R131.2
- new net S58: R132.2
- new net S59: R133.2
- new net S60: R134.2
- new net S61: R135.2
- new net S62: R136.2
- new net S63: R137.2
- new net S64: R162.2
- new net S65: R204.2
- new net S66: R205.2
- new net S67: R206.2
- new net S68: R207.2
- new net S69: R208.2
- new net S70: R209.2
- new net S71: R222.2
- new net S72: R223.2
- new net S73: R224.2
- new net S74: R225.2
- new net S75: R226.2
- new net S76: R227.2
- new net S77: R228.2
- new net S79: R246.2
- new net S80: R247.2
- new net S81: R248.2
- new net S82: R249.2
- new net S83: R250.2
- new net S84: R251.2
- new net S85: R252.2
- new net S86: R253.2
- new net S87: R271.2
- new net S88: R272.2
- new net S89: R273.2
- new net S90: R274.2
- new net S91: R275.2
- new net S92: R276.2
- new net S93: R277.2
- new net S94: R278.2
- new net S95: R295.2
- new net S96: R296.2
- new net S97: R297.2
- new net S98: R298.2
- new net S99: R299.2
- new net SOL100-: D93.2 (A), J101.2, Q92.5 (D_1), Q92.6 (D_2), Q92.7 (D_3), Q92.8 (D_4), Q92.9 (D_5)
- new net SOL101-: D94.2 (A), J102.2, Q93.5 (D_1), Q93.6 (D_2), Q93.7 (D_3), Q93.8 (D_4), Q93.9 (D_5)
- new net SOL102-: D95.2 (A), J105.2, Q94.5 (D_1), Q94.6 (D_2), Q94.7 (D_3), Q94.8 (D_4), Q94.9 (D_5)
- new net SOL103-: D96.2 (A), J110.2, Q95.5 (D_1), Q95.6 (D_2), Q95.7 (D_3), Q95.8 (D_4), Q95.9 (D_5)
- new net SOL104-: D97.2 (A), J108.2, Q96.5 (D_1), Q96.6 (D_2), Q96.7 (D_3), Q96.8 (D_4), Q96.9 (D_5)
- new net SOL105-: D98.2 (A), J106.2, Q97.5 (D_1), Q97.6 (D_2), Q97.7 (D_3), Q97.8 (D_4), Q97.9 (D_5)
- new net SOL106-: D99.2 (A), J111.2, Q98.5 (D_1), Q98.6 (D_2), Q98.7 (D_3), Q98.8 (D_4), Q98.9 (D_5)
- new net SOL107-: D100.2 (A), J109.2, Q99.5 (D_1), Q99.6 (D_2), Q99.7 (D_3), Q99.8 (D_4), Q99.9 (D_5)
- new net SOL108-: D109.2 (A), J107.2, Q100.5 (D_1), Q100.6 (D_2), Q100.7 (D_3), Q100.8 (D_4), Q100.9 (D_5)
- new net SOL109-: D110.2 (A), J112.2, Q109.5 (D_1), Q109.6 (D_2), Q109.7 (D_3), Q109.8 (D_4), Q109.9 (D_5)
- new net SOL110-: D111.2 (A), J113.2, Q110.5 (D_1), Q110.6 (D_2), Q110.7 (D_3), Q110.8 (D_4), Q110.9 (D_5)
- new net SOL119-: D120.2 (A), J126.2, Q119.5 (D_1), Q119.6 (D_2), Q119.7 (D_3), Q119.8 (D_4), Q119.9 (D_5)
- new net SOL120-: D121.2 (A), J124.2, Q120.5 (D_1), Q120.6 (D_2), Q120.7 (D_3), Q120.8 (D_4), Q120.9 (D_5)
- new net SOL121-: D122.2 (A), J122.2, Q121.5 (D_1), Q121.6 (D_2), Q121.7 (D_3), Q121.8 (D_4), Q121.9 (D_5)
- new net SOL122-: D123.2 (A), J127.2, Q122.5 (D_1), Q122.6 (D_2), Q122.7 (D_3), Q122.8 (D_4), Q122.9 (D_5)
- new net SOL123-: D124.2 (A), J125.2, Q123.5 (D_1), Q123.6 (D_2), Q123.7 (D_3), Q123.8 (D_4), Q123.9 (D_5)
- new net SOL124-: D125.2 (A), J123.2, Q124.5 (D_1), Q124.6 (D_2), Q124.7 (D_3), Q124.8 (D_4), Q124.9 (D_5)
- new net SOL125-: D126.2 (A), J128.2, Q125.5 (D_1), Q125.6 (D_2), Q125.7 (D_3), Q125.8 (D_4), Q125.9 (D_5)
- new net SOL126-: D127.2 (A), J129.2, Q126.5 (D_1), Q126.6 (D_2), Q126.7 (D_3), Q126.8 (D_4), Q126.9 (D_5)
- new net SOL127-: D128.2 (A), J132.2, Q127.5 (D_1), Q127.6 (D_2), Q127.7 (D_3), Q127.8 (D_4), Q127.9 (D_5)
- new net SOL128-: D129.2 (A), J133.2, Q128.5 (D_1), Q128.6 (D_2), Q128.7 (D_3), Q128.8 (D_4), Q128.9 (D_5)
- new net SOL129-: D130.2 (A), J134.2, Q129.5 (D_1), Q129.6 (D_2), Q129.7 (D_3), Q129.8 (D_4), Q129.9 (D_5)
- new net SOL130-: D131.2 (A), J130.2, Q130.5 (D_1), Q130.6 (D_2), Q130.7 (D_3), Q130.8 (D_4), Q130.9 (D_5)
- new net SOL131-: D132.2 (A), J135.2, Q131.5 (D_1), Q131.6 (D_2), Q131.7 (D_3), Q131.8 (D_4), Q131.9 (D_5)
- new net SOL132-: D133.2 (A), J136.2, Q132.5 (D_1), Q132.6 (D_2), Q132.7 (D_3), Q132.8 (D_4), Q132.9 (D_5)
- new net SOL133-: D134.2 (A), J131.2, Q133.5 (D_1), Q133.6 (D_2), Q133.7 (D_3), Q133.8 (D_4), Q133.9 (D_5)
- new net SOL134-: D135.2 (A), J137.2, Q134.5 (D_1), Q134.6 (D_2), Q134.7 (D_3), Q134.8 (D_4), Q134.9 (D_5)
- new net SOL135-: D136.2 (A), J139.2, Q135.5 (D_1), Q135.6 (D_2), Q135.7 (D_3), Q135.8 (D_4), Q135.9 (D_5)
- new net SOL136-: D137.2 (A), J140.2, Q136.5 (D_1), Q136.6 (D_2), Q136.7 (D_3), Q136.8 (D_4), Q136.9 (D_5)
- new net SOL137-: D138.2 (A), J141.2, Q137.5 (D_1), Q137.6 (D_2), Q137.7 (D_3), Q137.8 (D_4), Q137.9 (D_5)
- new net SOL138-: D139.2 (A), J138.2, Q138.5 (D_1), Q138.6 (D_2), Q138.7 (D_3), Q138.8 (D_4), Q138.9 (D_5)
- new net SOL139-: D140.2 (A), J142.2, Q139.5 (D_1), Q139.6 (D_2), Q139.7 (D_3), Q139.8 (D_4), Q139.9 (D_5)
- new net SOL140-: D141.2 (A), J143.2, Q140.5 (D_1), Q140.6 (D_2), Q140.7 (D_3), Q140.8 (D_4), Q140.9 (D_5)
- new net SOL49-: D42.2 (A), J6.2, Q41.5 (D_1), Q41.6 (D_2), Q41.7 (D_3), Q41.8 (D_4), Q41.9 (D_5)
- new net SOL50-: D43.2 (A), J4.2, Q42.5 (D_1), Q42.6 (D_2), Q42.7 (D_3), Q42.8 (D_4), Q42.9 (D_5)
- new net SOL51-: D44.2 (A), J1.2, Q43.5 (D_1), Q43.6 (D_2), Q43.7 (D_3), Q43.8 (D_4), Q43.9 (D_5)
- new net SOL52-: D45.2 (A), J7.2, Q44.5 (D_1), Q44.6 (D_2), Q44.7 (D_3), Q44.8 (D_4), Q44.9 (D_5)
- new net SOL53-: D46.2 (A), J5.2, Q45.5 (D_1), Q45.6 (D_2), Q45.7 (D_3), Q45.8 (D_4), Q45.9 (D_5)
- new net SOL54-: D47.2 (A), J2.2, Q46.5 (D_1), Q46.6 (D_2), Q46.7 (D_3), Q46.8 (D_4), Q46.9 (D_5)
- new net SOL55-: D48.2 (A), J56.2, Q47.5 (D_1), Q47.6 (D_2), Q47.7 (D_3), Q47.8 (D_4), Q47.9 (D_5)
- new net SOL56-: D49.2 (A), J57.2, Q48.5 (D_1), Q48.6 (D_2), Q48.7 (D_3), Q48.8 (D_4), Q48.9 (D_5)
- new net SOL57-: D50.2 (A), J60.2, Q49.5 (D_1), Q49.6 (D_2), Q49.7 (D_3), Q49.8 (D_4), Q49.9 (D_5)
- new net SOL58-: D51.2 (A), J61.2, Q50.5 (D_1), Q50.6 (D_2), Q50.7 (D_3), Q50.8 (D_4), Q50.9 (D_5)
- new net SOL59-: D52.2 (A), J62.2, Q51.5 (D_1), Q51.6 (D_2), Q51.7 (D_3), Q51.8 (D_4), Q51.9 (D_5)
- new net SOL60-: D53.2 (A), J58.2, Q52.5 (D_1), Q52.6 (D_2), Q52.7 (D_3), Q52.8 (D_4), Q52.9 (D_5)
- new net SOL61-: D54.2 (A), J63.2, Q53.5 (D_1), Q53.6 (D_2), Q53.7 (D_3), Q53.8 (D_4), Q53.9 (D_5)
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