File: NozzleControlBoard.kicad_sch (KiCad schematic)
At the start: 1139 parts, among them IC2 MAX3094EESE+, IC3 MAX22245BAWA+, J1 SOL51, J10 SOL3, J100 SOL99, J101 SOL100, J102 SOL101, J103 SHIFT_DATA_TOSS, J104 8BIT_24V_OUT, J105 SOL102, J106 SOL105, J107 SOL108, J108 SOL104, J109 SOL107, J11 SOL4, J110 SOL103, J111 SOL106, J112 SOL109, J113 SOL110, J114 SOL44, J115 SOL47, J116 SOL41, J117 SOL42, J118 SOL43, J119 SOL45, J12 SOL5, J120 SOL46, J121 SOL48, J122 SOL121, J123 SOL124, J124 SOL120, J125 SOL123, J126 SOL119, J127 SOL122, J128 SOL125, J129 SOL126, J13 SOL6, J130 SOL130, J131 SOL133, J132 SOL127, J133 SOL128, J134 SOL129, J135 SOL131, J136 SOL132, J137 SOL134, J138 SOL138, J139 SOL135, J14 SOL7, J140 SOL136, J141 SOL137, J142 SOL139, J143 SOL140, J144 SHIFT_DATA_TOSS, J145 8BIT_24V_OUT, J15 SOL8, J16 SOL9, J17 SOL10, J18 SOL11, J19 SOL12, J2 SOL54, J20 SOL13, J21 SOL14, J22 SOL15, J23 SOL16, J24 SOL17, J25 SOL18, J26 SOL19, J27 SOL20, J28 SOL21, J29 SOL22, J3 Conn_01x12_Male, J30 SOL23, J31 SOL24, J32 SOL25, J33 SOL26, J34 SOL27, J35 SOL28, J36 SOL29, J37 SOL30, J38 SOL31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

Commit message: 이은혜
4/1
Parts:
- J114: value SOL44 -> SOL114
- J115: value SOL47 -> SOL117
- J116: value SOL41 -> SOL111
- J117: value SOL42 -> SOL112
- J118: value SOL43 -> SOL113
- J119: value SOL45 -> SOL115
- J120: value SOL46 -> SOL116
- J121: value SOL48 -> SOL118
Connections:
- net S1: no longer U86.15 (QA)
- net S10: no longer U95.1 (QB)
- net S100: now also U123.5 (QF)
- net S101: now also U123.6 (QG)
- net S102: now also U123.7 (QH)
- net S103: now also U133.15 (QA)
- net S104: now also U133.1 (QB)
- net S105: now also U133.2 (QC)
- net S106: now also U133.3 (QD)
- net S107: now also U133.4 (QE)
- net S108: now also U133.5 (QF)
- net S109: now also U133.6 (QG)
- net S11: no longer U95.2 (QC)
- net S110: now also U133.7 (QH)
- net S111: now also U142.15 (QA)
- net S112: now also U142.1 (QB)
- net S113: now also U142.2 (QC)
- net S114: now also U142.3 (QD)
- net S115: now also U142.4 (QE)
- net S116: now also U142.5 (QF)
- net S117: now also U142.6 (QG)
- net S118: now also U142.7 (QH)
- net S119: now also U152.15 (QA)
- net S12: no longer U95.3 (QD)
- net S120: now also U152.1 (QB)
- net S121: now also U152.2 (QC)
- net S122: now also U152.3 (QD)
- net S123: now also U152.4 (QE)
- net S124: now also U152.5 (QF)
- net S125: now also U152.6 (QG)
- net S126: now also U152.7 (QH)
- net S127: now also U161.15 (QA)
- net S128: now also U161.1 (QB)
- net S129: now also U161.2 (QC)
- net S13: no longer U95.4 (QE)
- net S130: now also U161.3 (QD)
- net S131: now also U161.4 (QE)
- net S132: now also U161.5 (QF)
- net S133: now also U161.6 (QG)
- net S134: now also U161.7 (QH)
- net S135: now also U168.15 (QA)
- net S136: now also U168.1 (QB)
- net S137: now also U168.2 (QC)
- net S138: now also U168.3 (QD)
- net S139: now also U168.4 (QE)
- net S14: no longer U95.5 (QF)
- net S140: now also U168.5 (QF)
- net S15: no longer U95.6 (QG)
- net S16: no longer U95.7 (QH)
- net S17: no longer U114.15 (QA)
- net S18: no longer U114.1 (QB)
- net S19: no longer U114.2 (QC)
- net S2: no longer U86.1 (QB)
- net S20: no longer U114.3 (QD)
- net S21: no longer U114.4 (QE)
- net S22: no longer U114.5 (QF)
- net S23: no longer U114.6 (QG)
- net S24: no longer U114.7 (QH)
- net S25: no longer U123.15 (QA)
- net S26: no longer U123.1 (QB)
- net S27: no longer U123.2 (QC)
- net S28: no longer U123.3 (QD)
- net S29: no longer U123.4 (QE)
- net S3: no longer U86.2 (QC)
- net S30: no longer U123.5 (QF)
- net S31: no longer U123.6 (QG)
- net S32: no longer U123.7 (QH)
- net S33: no longer U133.15 (QA), U152.15 (QA), U37.15 (QA)
- net S34: no longer U133.1 (QB), U152.1 (QB), U37.1 (QB)
- net S35: no longer U133.2 (QC), U152.2 (QC), U37.2 (QC)
- net S36: no longer U133.3 (QD), U152.3 (QD), U37.3 (QD)
- net S37: no longer U133.4 (QE), U152.4 (QE), U37.4 (QE)
- net S38: no longer U133.5 (QF), U152.5 (QF), U37.5 (QF)
- net S39: no longer U133.6 (QG), U152.6 (QG), U37.6 (QG)
- net S4: no longer U86.3 (QD)
- net S40: no longer U133.7 (QH), U152.7 (QH), U37.7 (QH)
- net S41: no longer U142.15 (QA), U161.15 (QA), U168.15 (QA), U51.15 (QA), U68.15 (QA)
- net S42: no longer U142.1 (QB), U161.1 (QB), U168.1 (QB), U51.1 (QB), U68.1 (QB)
- net S43: no longer U142.2 (QC), U161.2 (QC), U168.2 (QC), U51.2 (QC), U68.2 (QC)
- net S44: no longer U142.3 (QD), U161.3 (QD), U168.3 (QD), U51.3 (QD), U68.3 (QD)
- net S45: no longer U142.4 (QE), U161.4 (QE), U168.4 (QE), U51.4 (QE), U68.4 (QE)
- net S46: no longer U142.5 (QF), U161.5 (QF), U168.5 (QF), U51.5 (QF), U68.5 (QF)
- net S47: no longer U142.6 (QG), U161.6 (QG), U168.6 (QG), U51.6 (QG), U68.6 (QG)
- net S48: no longer U142.7 (QH), U161.7 (QH), U168.7 (QH), U51.7 (QH), U68.7 (QH)
- net S49: now also U37.15 (QA)
- net S5: no longer U86.4 (QE)
- net S50: now also U37.1 (QB)
- net S51: now also U37.2 (QC)
- net S52: now also U37.3 (QD)
- net S53: now also U37.4 (QE)
- net S54: now also U37.5 (QF)
- net S55: now also U37.6 (QG)
- net S56: now also U37.7 (QH)
- net S57: now also U51.15 (QA)
- net S58: now also U51.1 (QB)
- net S59: now also U51.2 (QC)
- net S6: no longer U86.5 (QF)
- net S60: now also U51.3 (QD)
- net S61: now also U51.4 (QE)
- net S62: now also U51.5 (QF)
- net S63: now also U51.6 (QG)
- net S64: now also U51.7 (QH)
- net S65: now also U68.15 (QA)
- net S66: now also U68.1 (QB)
- net S67: now also U68.2 (QC)
- net S68: now also U68.3 (QD)
- net S69: now also U68.4 (QE)
- net S7: no longer U86.6 (QG)
- net S70: now also U68.5 (QF)
- net S71: now also U86.15 (QA)
- net S72: now also U86.1 (QB)
- net S73: now also U86.2 (QC)
- net S74: now also U86.3 (QD)
- net S75: now also U86.4 (QE)
- net S76: now also U86.5 (QF)
- net S77: now also U86.6 (QG)
- net S79: now also U95.15 (QA)
- net S8: no longer U86.7 (QH)
- net S80: now also U95.1 (QB)
- net S81: now also U95.2 (QC)
- net S82: now also U95.3 (QD)
- net S83: now also U95.4 (QE)
- net S84: now also U95.5 (QF)
- net S85: now also U95.6 (QG)
- net S86: now also U95.7 (QH)
- net S87: now also U114.15 (QA)
- net S88: now also U114.1 (QB)
- net S89: now also U114.2 (QC)
- net S9: no longer U95.15 (QA)
- net S90: now also U114.3 (QD)
- net S91: now also U114.4 (QE)
- net S92: now also U114.5 (QF)
- net S93: now also U114.6 (QG)
- net S94: now also U114.7 (QH)
- net S95: now also U123.15 (QA)
- net S96: now also U123.1 (QB)
- net S97: now also U123.2 (QC)
- net S98: now also U123.3 (QD)
- net S99: now also U123.4 (QE)
- net SOL41-: no longer D112.2 (A), J116.2, Q111.5 (D_1), Q111.6 (D_2), Q111.7 (D_3), Q111.8 (D_4), Q111.9 (D_5)
- net SOL42-: no longer D113.2 (A), J117.2, Q112.5 (D_1), Q112.6 (D_2), Q112.7 (D_3), Q112.8 (D_4), Q112.9 (D_5)
- net SOL43-: no longer D114.2 (A), J118.2, Q113.5 (D_1), Q113.6 (D_2), Q113.7 (D_3), Q113.8 (D_4), Q113.9 (D_5)
- net SOL44-: no longer D115.2 (A), J114.2, Q114.5 (D_1), Q114.6 (D_2), Q114.7 (D_3), Q114.8 (D_4), Q114.9 (D_5)
- net SOL45-: no longer D116.2 (A), J119.2, Q115.5 (D_1), Q115.6 (D_2), Q115.7 (D_3), Q115.8 (D_4), Q115.9 (D_5)
- net SOL46-: no longer D117.2 (A), J120.2, Q116.5 (D_1), Q116.6 (D_2), Q116.7 (D_3), Q116.8 (D_4), Q116.9 (D_5)
- net SOL47-: no longer D118.2 (A), J115.2, Q117.5 (D_1), Q117.6 (D_2), Q117.7 (D_3), Q117.8 (D_4), Q117.9 (D_5)
- net SOL48-: no longer D119.2 (A), J121.2, Q118.5 (D_1), Q118.6 (D_2), Q118.7 (D_3), Q118.8 (D_4), Q118.9 (D_5)
- new net S: U168.6 (QG), U168.7 (QH), U68.6 (QG), U68.7 (QH)
- new net S78: U86.7 (QH)
- new net SOL111-: D112.2 (A), J116.2, Q111.5 (D_1), Q111.6 (D_2), Q111.7 (D_3), Q111.8 (D_4), Q111.9 (D_5)
- new net SOL112-: D113.2 (A), J117.2, Q112.5 (D_1), Q112.6 (D_2), Q112.7 (D_3), Q112.8 (D_4), Q112.9 (D_5)
- new net SOL113-: D114.2 (A), J118.2, Q113.5 (D_1), Q113.6 (D_2), Q113.7 (D_3), Q113.8 (D_4), Q113.9 (D_5)
- new net SOL114-: D115.2 (A), J114.2, Q114.5 (D_1), Q114.6 (D_2), Q114.7 (D_3), Q114.8 (D_4), Q114.9 (D_5)
- new net SOL115-: D116.2 (A), J119.2, Q115.5 (D_1), Q115.6 (D_2), Q115.7 (D_3), Q115.8 (D_4), Q115.9 (D_5)
- new net SOL116-: D117.2 (A), J120.2, Q116.5 (D_1), Q116.6 (D_2), Q116.7 (D_3), Q116.8 (D_4), Q116.9 (D_5)
- new net SOL117-: D118.2 (A), J115.2, Q117.5 (D_1), Q117.6 (D_2), Q117.7 (D_3), Q117.8 (D_4), Q117.9 (D_5)
- new net SOL118-: D119.2 (A), J121.2, Q118.5 (D_1), Q118.6 (D_2), Q118.7 (D_3), Q118.8 (D_4), Q118.9 (D_5)

Commit message: 이은혜
4/2
Parts:
- Q66: footprint TPN22006NH:TPN22006NHLQ -> footprint:TPN22006NHLQ
Changed lines of the file:
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@@
       (effects (font (size 1.27 1.27)))
     )
-    (property "Footprint" "TPN22006NH:TPN22006NHLQ" (at 766.445 643.255 0)
+    (property "Footprint" "footprint:TPN22006NHLQ" (at 766.445 643.255 0)
       (effects (font (size 1.27 1.27)) (justify left) hide)
     )
