File: NozzleControlBoard.kicad_sch (KiCad schematic)
At the start: 1139 parts, among them IC2 MAX3094EESE+, IC3 MAX22245BAWA+, J1 SOL51, J10 SOL3, J100 SOL99, J101 SOL100, J102 SOL101, J103 SHIFT_DATA_TOSS, J104 8BIT_24V_OUT, J105 SOL102, J106 SOL105, J107 SOL108, J108 SOL104, J109 SOL107, J11 SOL4, J110 SOL103, J111 SOL106, J112 SOL109, J113 SOL110, J114 SOL114, J115 SOL117, J116 SOL111, J117 SOL112, J118 SOL113, J119 SOL115, J12 SOL5, J120 SOL116, J121 SOL118, J122 SOL121, J123 SOL124, J124 SOL120, J125 SOL123, J126 SOL119, J127 SOL122, J128 SOL125, J129 SOL126, J13 SOL6, J130 SOL130, J131 SOL133, J132 SOL127, J133 SOL128, J134 SOL129, J135 SOL131, J136 SOL132, J137 SOL134, J138 SOL138, J139 SOL135, J14 SOL7, J140 SOL136, J141 SOL137, J142 SOL139, J143 SOL140, J144 SHIFT_DATA_TOSS, J145 8BIT_24V_OUT, J15 SOL8, J16 SOL9, J17 SOL10, J18 SOL11, J19 SOL12, J2 SOL54, J20 SOL13, J21 SOL14, J22 SOL15, J23 SOL16, J24 SOL17, J25 SOL18, J26 SOL19, J27 SOL20, J28 SOL21, J29 SOL22, J3 Conn_01x12_Male, J30 SOL23, J31 SOL24, J32 SOL25, J33 SOL26, J34 SOL27, J35 SOL28, J36 SOL29, J37 SOL30, J38 SOL31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

Commit message: .
.
Parts:
- added R436, R437, R438, R439, R440, R441, R442, R443, R444, R445, R446, R447, R448, R449, R450, R451, R452, R453, R454, R455, R456, R457, R458, R459, R460, R461, R462, R463, R464, R465, R466, R467, R468, R469, R470, R471, R472, R473, R474, R475, R476, R477, R478, R479, R480, R481, R482, R483, R484, R485, R486, R487, R488, R489, R490, R491, R492, R493, R494, R495, R496, R497, R498, R499, R500, R501, R502, R503, R504, R505, R506, R507, R508, R509, R510, R511, R512, R513, R514, R515, R516, R517, R518, R519, R520, R521, R522, R523, R524, R525, R526, R527, R528, R529, R530, R531, R532, R533, R534, R535, R536, R537, R538, R539, R540, R541, R542, R543, R544, R545, R546, R547, R548, R549, R550, R551, R552, R553, R554, R555, R556, R557, R558, R559, R560, R561, R562, R563, R564, R565, R566, R567, R568, R569, R570, R571, R572, R573, R574, R575: 1.2k, Resistor_SMD:R_1206_3216Metric_Pad1.30x1.75mm_HandSolder, symbol Device:R
- added U170, U172, U175, U177, U179: FFC_60PIN_UP, FFC_60_PIN:FFC_60PIN, symbol FFC_60PIN_UP:FFC_60PIN_UP
Connections:
- new net 24V: U170.1, U170.2, U170.3, U170.4, U170.5, U170.6, U172.1, U172.2, U172.3, U172.4, U172.5, U172.6
- new net 24V_2: U175.1, U175.2, U175.3, U175.4, U175.5, U175.6, U177.1, U177.2, U177.3, U177.4, U177.5, U177.6, U179.1, U179.2, U179.3, U179.4, U179.5, U179.6
- new net CH1: R467.1
- new net CH10: R458.1
- new net CH100: R560.1
- new net CH101: R559.1
- new net CH102: R558.1
- new net CH103: R557.1
- new net CH104: R556.1
- new net CH105: R555.1
- new net CH106: R554.1
- new net CH107: R553.1
- new net CH108: R552.1
- new net CH109: R551.1
- new net CH11: R457.1
- new net CH110: R550.1
- new net CH111: R549.1
- new net CH112: R548.1
- new net CH113: R547.1
- new net CH114: R546.1
- new net CH115: R545.1
- new net CH116: R544.1
- new net CH117: R543.1
- new net CH118: R542.1
- new net CH119: R541.1
- new net CH12: R456.1
- new net CH120: R540.1
- new net CH121: R539.1
- new net CH122: R538.1
- new net CH123: R537.1
- new net CH124: R536.1
- new net CH125: R535.1
- new net CH126: R534.1
- new net CH127: R533.1
- new net CH128: R532.1
- new net CH129: R575.1
- new net CH13: R455.1
- new net CH130: R574.1
- new net CH131: R573.1
- new net CH132: R572.1
- new net CH133: R571.1
- new net CH134: R570.1
- new net CH135: R569.1
- new net CH136: R568.1
- new net CH137: R567.1
- new net CH138: R566.1
- new net CH139: R565.1
- new net CH14: R454.1
- new net CH140: R564.1
- new net CH15: R453.1
- new net CH16: R452.1
- new net CH17: R451.1
- new net CH18: R450.1
- new net CH19: R449.1
- new net CH2: R466.1
- new net CH20: R448.1
- new net CH21: R447.1
- new net CH22: R446.1
- new net CH23: R445.1
- new net CH24: R444.1
- new net CH25: R443.1
- new net CH26: R442.1
- new net CH27: R441.1
- new net CH28: R440.1
- new net CH29: R439.1
- new net CH3: R465.1
- new net CH30: R438.1
- new net CH31: R437.1
- new net CH32: R436.1
- new net CH33: R499.1
- new net CH34: R498.1
- new net CH35: R497.1
- new net CH36: R496.1
- new net CH37: R495.1
- new net CH38: R494.1
- new net CH39: R493.1
- new net CH4: R464.1
- new net CH40: R492.1
- new net CH41: R491.1
- new net CH42: R490.1
- new net CH43: R489.1
- new net CH44: R488.1
- new net CH45: R487.1
- new net CH46: R486.1
- new net CH47: R485.1
- new net CH48: R484.1
- new net CH49: R483.1
- new net CH5: R463.1
- new net CH50: R482.1
- new net CH51: R481.1
- new net CH52: R480.1
- new net CH53: R479.1
- new net CH54: R478.1
- new net CH55: R477.1
- new net CH56: R476.1
- new net CH57: R475.1
- new net CH58: R474.1
- new net CH59: R473.1
- new net CH6: R462.1
- new net CH60: R472.1
- new net CH61: R471.1
- new net CH62: R470.1
- new net CH63: R469.1
- new net CH64: R468.1
- new net CH65: R531.1
- new net CH66: R530.1
- new net CH67: R529.1
- new net CH68: R528.1
- new net CH69: R527.1
- new net CH7: R461.1
- new net CH70: R526.1
- new net CH71: R525.1
- new net CH72: R524.1
- new net CH73: R523.1
- new net CH74: R522.1
- new net CH75: R521.1
- new net CH76: R520.1
- new net CH77: R519.1
- new net CH78: R518.1
- new net CH79: R517.1
- new net CH8: R460.1
- new net CH80: R516.1
- new net CH81: R515.1
- new net CH82: R514.1
- new net CH83: R513.1
- new net CH84: R512.1
- new net CH85: R511.1
- new net CH86: R510.1
- new net CH87: R509.1
- new net CH88: R508.1
- new net CH89: R507.1
- new net CH9: R459.1
- new net CH90: R506.1
- new net CH91: R505.1
- new net CH92: R504.1
- new net CH93: R503.1
- new net CH94: R502.1
- new net CH95: R501.1
- new net CH96: R500.1
- new net CH97: R563.1
- new net CH98: R562.1
- new net CH99: R561.1
- new net GND: U170.17, U170.18, U170.19, U170.20, U170.21, U170.22, U172.17, U172.18, U172.19, U172.20, U172.21, U172.22
- new net GND_2: U175.17, U175.18, U175.19, U175.20, U175.21, U175.22, U177.17, U177.18, U177.19, U177.20, U177.21, U177.22, U179.17, U179.18, U179.19, U179.20, U179.21, U179.22
- new net LED1: R467.2, U170.60
- new net LED10: R458.2, U170.51
- new net LED100: R560.2, U177.57
- new net LED101: R559.2, U177.56
- new net LED102: R558.2, U177.55
- new net LED103: R557.2, U177.54
- new net LED104: R556.2, U177.53
- new net LED105: R555.2, U177.52
- new net LED106: R554.2, U177.51
- new net LED107: R553.2, U177.50
- new net LED108: R552.2, U177.49
- new net LED109: R551.2, U177.48
- new net LED11: R457.2, U170.50
- new net LED110: R550.2, U177.47
- new net LED111: R549.2, U177.46
- new net LED112: R548.2, U177.45
- new net LED113: R547.2, U177.44
- new net LED114: R546.2, U177.43
- new net LED115: R545.2, U177.42
- new net LED116: R544.2, U177.41
- new net LED117: R543.2, U177.40
- new net LED118: R542.2, U177.39
- new net LED119: R541.2, U177.38
- new net LED12: R456.2, U170.49
- new net LED120: R540.2, U177.37
- new net LED121: R539.2, U177.36
- new net LED122: R538.2, U177.35
- new net LED123: R537.2, U177.34
- new net LED124: R536.2, U177.33
- new net LED125: R535.2, U177.32
- new net LED126: R534.2, U177.31
- new net LED127: R533.2, U177.30
- new net LED128: R532.2, U177.29
- new net LED129: R575.2, U179.60
- new net LED13: R455.2, U170.48
- new net LED130: R574.2, U179.59
- new net LED131: R573.2, U179.58
- new net LED132: R572.2, U179.57
- new net LED133: R571.2, U179.56
- new net LED134: R570.2, U179.55
- new net LED135: R569.2, U179.54
- new net LED136: R568.2, U179.53
- new net LED137: R567.2, U179.52
- new net LED138: R566.2, U179.51
- new net LED139: R565.2, U179.50
- new net LED14: R454.2, U170.47
- new net LED140: R564.2, U179.49
- new net LED15: R453.2, U170.46
- new net LED16: R452.2, U170.45
- new net LED17: R451.2, U170.44
- new net LED18: R450.2, U170.43
- new net LED19: R449.2, U170.42
- new net LED2: R466.2, U170.59
- new net LED20: R448.2, U170.41
- new net LED21: R447.2, U170.40
- new net LED22: R446.2, U170.39
- new net LED23: R445.2, U170.38
- new net LED24: R444.2, U170.37
- new net LED25: R443.2, U170.36
- new net LED26: R442.2, U170.35
- new net LED27: R441.2, U170.34
- new net LED28: R440.2, U170.33
- new net LED29: R439.2, U170.32
- new net LED3: R465.2, U170.58
- new net LED30: R438.2, U170.31
- new net LED31: R437.2, U170.30
- new net LED32: R436.2, U170.29
- new net LED33: R499.2, U172.60
- new net LED34: R498.2, U172.59
- new net LED35: R497.2, U172.58
- new net LED36: R496.2, U172.57
- new net LED37: R495.2, U172.56
- new net LED38: R494.2, U172.55
- new net LED39: R493.2, U172.54
- new net LED4: R464.2, U170.57
- new net LED40: R492.2, U172.53
- new net LED41: R491.2, U172.52
- new net LED42: R490.2, U172.51
- new net LED43: R489.2, U172.50
- new net LED44: R488.2, U172.49
- new net LED45: R487.2, U172.48
- new net LED46: R486.2, U172.47
- new net LED47: R485.2, U172.46
- new net LED48: R484.2, U172.45
- new net LED49: R483.2, U172.44
- new net LED5: R463.2, U170.56
- new net LED50: R482.2, U172.43
- new net LED51: R481.2, U172.42
- new net LED52: R480.2, U172.41
- new net LED53: R479.2, U172.40
- new net LED54: R478.2, U172.39
- new net LED55: R477.2, U172.38
- new net LED56: R476.2, U172.37
- new net LED57: R475.2, U172.36
- new net LED58: R474.2, U172.35
- new net LED59: R473.2, U172.34
- new net LED6: R462.2, U170.55
- new net LED60: R472.2, U172.33
- new net LED61: R471.2, U172.32
- new net LED62: R470.2, U172.31
- new net LED63: R469.2, U172.30
- new net LED64: R468.2, U172.29
- new net LED65: R531.2, U175.60
- new net LED66: R530.2, U175.59
- new net LED67: R529.2, U175.58
- new net LED68: R528.2, U175.57
- new net LED69: R527.2, U175.56
- new net LED7: R461.2, U170.54
- new net LED70: R526.2, U175.55
- new net LED71: R525.2, U175.54
- new net LED72: R524.2, U175.53
- new net LED73: R523.2, U175.52
- new net LED74: R522.2, U175.51
- new net LED75: R521.2, U175.50
- new net LED76: R520.2, U175.49
- new net LED77: R519.2, U175.48
- new net LED78: R518.2, U175.47
- new net LED79: R517.2, U175.46
- new net LED8: R460.2, U170.53
- new net LED80: R516.2, U175.45
- new net LED81: R515.2, U175.44
- new net LED82: R514.2, U175.43
- new net LED83: R513.2, U175.42
- new net LED84: R512.2, U175.41
- new net LED85: R511.2, U175.40
- new net LED86: R510.2, U175.39
- new net LED87: R509.2, U175.38
- new net LED88: R508.2, U175.37
- new net LED89: R507.2, U175.36
- new net LED9: R459.2, U170.52
- new net LED90: R506.2, U175.35
- new net LED91: R505.2, U175.34
- new net LED92: R504.2, U175.33
- new net LED93: R503.2, U175.32
- new net LED94: R502.2, U175.31
- new net LED95: R501.2, U175.30
- new net LED96: R500.2, U175.29
- new net LED97: R563.2, U177.60
- new net LED98: R562.2, U177.59
- new net LED99: R561.2, U177.58

Commit message: 이은혜
Connections:
- net SOL1- is gone; now on net CH1: D1.2 (A), J8.2, Q1.5 (D_1), Q1.6 (D_2), Q1.7 (D_3), Q1.8 (D_4), Q1.9 (D_5)
Changed lines of the file:
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@@
   (junction (at 1105.535 321.945) (diameter 0) (color 0 0 0 0)
   )
+  (junction (at 798.83 132.715) (diameter 0) (color 0 0 0 0)
+  )
   (junction (at 1265.555 632.46) (diameter 0) (color 0 0 0 0)
   )
@@
     (stroke (width 0) (type default))
   )
+  (wire (pts (xy 798.83 140.97) (xy 798.83 132.715))
+    (stroke (width 0) (type default))
+  )
   (wire (pts (xy 1931.035 363.855) (xy 1942.465 363.855))
     (stroke (width 0) (type default))
@@
     (stroke (width 0) (type default))
   )
+  (wire (pts (xy 798.83 140.97) (xy 807.72 140.97))
+    (stroke (width 0) (type default))
+  )
   (wire (pts (xy 1469.1476 721.36) (xy 1489.71 721.36))
     (stroke (width 0) (type default))
@@
     (stroke (width 0) (type default))
   )
-  (wire (pts (xy 780.1726 132.715) (xy 800.735 132.715))
-    (stroke (width 0) (type default))
-  )
   (wire (pts (xy 909.955 648.335) (xy 909.955 645.795))
     (stroke (width 0) (type default))
@@
     (stroke (width 0) (type default))
   )
+  (wire (pts (xy 798.83 132.715) (xy 800.735 132.715))
+    (stroke (width 0) (type default))
+  )
   (polyline (pts (xy 271.78 82.55) (xy 528.32 82.55))
     (stroke (width 1) (type solid) (color 255 136 6 1))
@@
     (stroke (width 0) (type default))
   )
+  (wire (pts (xy 780.1726 132.715) (xy 798.83 132.715))
+    (stroke (width 0) (type default))
+  )
   (wire (pts (xy 2739.39 252.73) (xy 2731.77 252.73))
     (stroke (width 0) (type default))
@@
     (effects (font (size 1.27 1.27)) (justify left bottom))
   )
+  (label "CH1" (at 801.37 140.97 0) (fields_autoplaced)
+    (effects (font (size 1.27 1.27)) (justify left bottom))
+  )

Commit message: 이은혜
4/7 32CH 확인해주세요
Parts:
- Q4: footprint TPN22006NH:TPN22006NHLQ -> footprint:TPN22006NHLQ
Connections:
- net SOL10- is gone; now on net CH10: D11.2 (A), J17.2, Q10.5 (D_1), Q10.6 (D_2), Q10.7 (D_3), Q10.8 (D_4), Q10.9 (D_5)
- net SOL11- is gone; now on net CH11: D12.2 (A), J18.2, Q11.5 (D_1), Q11.6 (D_2), Q11.7 (D_3), Q11.8 (D_4), Q11.9 (D_5)
- net SOL12- is gone; now on net CH12: D13.2 (A), J19.2, Q12.5 (D_1), Q12.6 (D_2), Q12.7 (D_3), Q12.8 (D_4), Q12.9 (D_5)
- net SOL13- is gone; now on net CH13: D14.2 (A), J20.2, Q13.5 (D_1), Q13.6 (D_2), Q13.7 (D_3), Q13.8 (D_4), Q13.9 (D_5)
- net SOL14- is gone; now on net CH14: D15.2 (A), J21.2, Q14.5 (D_1), Q14.6 (D_2), Q14.7 (D_3), Q14.8 (D_4), Q14.9 (D_5)
- net SOL15- is gone; now on net CH15: D16.2 (A), J22.2, Q15.5 (D_1), Q15.6 (D_2), Q15.7 (D_3), Q15.8 (D_4), Q15.9 (D_5)
- net SOL16- is gone; now on net CH16: D17.2 (A), J23.2, Q16.5 (D_1), Q16.6 (D_2), Q16.7 (D_3), Q16.8 (D_4), Q16.9 (D_5)
- net SOL17- is gone; now on net CH17: D18.2 (A), J24.2, Q17.5 (D_1), Q17.6 (D_2), Q17.7 (D_3), Q17.8 (D_4), Q17.9 (D_5)
- net SOL18- is gone; now on net CH18: D19.2 (A), J25.2, Q18.5 (D_1), Q18.6 (D_2), Q18.7 (D_3), Q18.8 (D_4), Q18.9 (D_5)
- net SOL19- is gone; now on net CH19: D20.2 (A), J26.2, Q19.5 (D_1), Q19.6 (D_2), Q19.7 (D_3), Q19.8 (D_4), Q19.9 (D_5)
- net SOL2- is gone; now on net CH2: D3.2 (A), J9.2, Q2.5 (D_1), Q2.6 (D_2), Q2.7 (D_3), Q2.8 (D_4), Q2.9 (D_5)
- net SOL20- is gone; now on net CH20: D21.2 (A), J27.2, Q20.5 (D_1), Q20.6 (D_2), Q20.7 (D_3), Q20.8 (D_4), Q20.9 (D_5)
- net SOL21- is gone; now on net CH21: D22.2 (A), J28.2, Q21.5 (D_1), Q21.6 (D_2), Q21.7 (D_3), Q21.8 (D_4), Q21.9 (D_5)
- net SOL22- is gone; now on net CH22: D23.2 (A), J29.2, Q22.5 (D_1), Q22.6 (D_2), Q22.7 (D_3), Q22.8 (D_4), Q22.9 (D_5)
- net SOL23- is gone; now on net CH23: D24.2 (A), J30.2, Q23.5 (D_1), Q23.6 (D_2), Q23.7 (D_3), Q23.8 (D_4), Q23.9 (D_5)
- net SOL24- is gone; now on net CH24: D25.2 (A), J31.2, Q24.5 (D_1), Q24.6 (D_2), Q24.7 (D_3), Q24.8 (D_4), Q24.9 (D_5)
- net SOL25- is gone; now on net CH25: D101.2 (A), J32.2, Q101.5 (D_1), Q101.6 (D_2), Q101.7 (D_3), Q101.8 (D_4), Q101.9 (D_5)
- net SOL26- is gone; now on net CH26: D102.2 (A), J33.2, Q102.5 (D_1), Q102.6 (D_2), Q102.7 (D_3), Q102.8 (D_4), Q102.9 (D_5)
- net SOL27- is gone; now on net CH27: D103.2 (A), J34.2, Q103.5 (D_1), Q103.6 (D_2), Q103.7 (D_3), Q103.8 (D_4), Q103.9 (D_5)
- net SOL28- is gone; now on net CH28: D104.2 (A), J35.2, Q104.5 (D_1), Q104.6 (D_2), Q104.7 (D_3), Q104.8 (D_4), Q104.9 (D_5)
- net SOL29- is gone; now on net CH29: D105.2 (A), J36.2, Q105.5 (D_1), Q105.6 (D_2), Q105.7 (D_3), Q105.8 (D_4), Q105.9 (D_5)
- net SOL3- is gone; now on net CH3: D4.2 (A), J10.2, Q3.5 (D_1), Q3.6 (D_2), Q3.7 (D_3), Q3.8 (D_4), Q3.9 (D_5)
- net SOL30- is gone; now on net CH30: D106.2 (A), J37.2, Q106.5 (D_1), Q106.6 (D_2), Q106.7 (D_3), Q106.8 (D_4), Q106.9 (D_5)
- net SOL31- is gone; now on net CH31: D107.2 (A), J38.2, Q107.5 (D_1), Q107.6 (D_2), Q107.7 (D_3), Q107.8 (D_4), Q107.9 (D_5)
- net SOL32- is gone; now on net CH32: D108.2 (A), J39.2, Q108.5 (D_1), Q108.6 (D_2), Q108.7 (D_3), Q108.8 (D_4), Q108.9 (D_5)
- net SOL4- is gone; now on net CH4: D5.2 (A), J11.2, Q4.5 (D_1), Q4.6 (D_2), Q4.7 (D_3), Q4.8 (D_4), Q4.9 (D_5)
- net SOL5- is gone; now on net CH5: D6.2 (A), J12.2, Q5.5 (D_1), Q5.6 (D_2), Q5.7 (D_3), Q5.8 (D_4), Q5.9 (D_5)
- net SOL6- is gone; now on net CH6: D7.2 (A), J13.2, Q6.5 (D_1), Q6.6 (D_2), Q6.7 (D_3), Q6.8 (D_4), Q6.9 (D_5)
- net SOL7- is gone; now on net CH7: D8.2 (A), J14.2, Q7.5 (D_1), Q7.6 (D_2), Q7.7 (D_3), Q7.8 (D_4), Q7.9 (D_5)
- net SOL8- is gone; now on net CH8: D9.2 (A), J15.2, Q8.5 (D_1), Q8.6 (D_2), Q8.7 (D_3), Q8.8 (D_4), Q8.9 (D_5)
- net SOL9- is gone; now on net CH9: D10.2 (A), J16.2, Q9.5 (D_1), Q9.6 (D_2), Q9.7 (D_3), Q9.8 (D_4), Q9.9 (D_5)

Commit message: 이은혜
....
Connections:
- net 78 is gone; now on net S78: R229.2
- net SOL100- is gone; now on net CH100: D93.2 (A), J101.2, Q92.5 (D_1), Q92.6 (D_2), Q92.7 (D_3), Q92.8 (D_4), Q92.9 (D_5)
- net SOL101- is gone; now on net CH101: D94.2 (A), J102.2, Q93.5 (D_1), Q93.6 (D_2), Q93.7 (D_3), Q93.8 (D_4), Q93.9 (D_5)
- net SOL102- is gone; now on net CH102: D95.2 (A), J105.2, Q94.5 (D_1), Q94.6 (D_2), Q94.7 (D_3), Q94.8 (D_4), Q94.9 (D_5)
- net SOL103- is gone; now on net CH103: D96.2 (A), J110.2, Q95.5 (D_1), Q95.6 (D_2), Q95.7 (D_3), Q95.8 (D_4), Q95.9 (D_5)
- net SOL104- is gone; now on net CH104: D97.2 (A), J108.2, Q96.5 (D_1), Q96.6 (D_2), Q96.7 (D_3), Q96.8 (D_4), Q96.9 (D_5)
- net SOL105- is gone; now on net CH105: D98.2 (A), J106.2, Q97.5 (D_1), Q97.6 (D_2), Q97.7 (D_3), Q97.8 (D_4), Q97.9 (D_5)
- net SOL106- is gone; now on net CH106: D99.2 (A), J111.2, Q98.5 (D_1), Q98.6 (D_2), Q98.7 (D_3), Q98.8 (D_4), Q98.9 (D_5)
- net SOL107- is gone; now on net CH107: D100.2 (A), J109.2, Q99.5 (D_1), Q99.6 (D_2), Q99.7 (D_3), Q99.8 (D_4), Q99.9 (D_5)
- net SOL108- is gone; now on net CH108: D109.2 (A), J107.2, Q100.5 (D_1), Q100.6 (D_2), Q100.7 (D_3), Q100.8 (D_4), Q100.9 (D_5)
- net SOL109- is gone; now on net CH109: D110.2 (A), J112.2, Q109.5 (D_1), Q109.6 (D_2), Q109.7 (D_3), Q109.8 (D_4), Q109.9 (D_5)
- net SOL110- is gone; now on net CH110: D111.2 (A), J113.2, Q110.5 (D_1), Q110.6 (D_2), Q110.7 (D_3), Q110.8 (D_4), Q110.9 (D_5)
- net SOL111- is gone; now on net CH111: D112.2 (A), J116.2, Q111.5 (D_1), Q111.6 (D_2), Q111.7 (D_3), Q111.8 (D_4), Q111.9 (D_5)
- net SOL112- is gone; now on net CH112: D113.2 (A), J117.2, Q112.5 (D_1), Q112.6 (D_2), Q112.7 (D_3), Q112.8 (D_4), Q112.9 (D_5)
- net SOL113- is gone; now on net CH113: D114.2 (A), J118.2, Q113.5 (D_1), Q113.6 (D_2), Q113.7 (D_3), Q113.8 (D_4), Q113.9 (D_5)
- net SOL114- is gone; now on net CH114: D115.2 (A), J114.2, Q114.5 (D_1), Q114.6 (D_2), Q114.7 (D_3), Q114.8 (D_4), Q114.9 (D_5)
- net SOL115- is gone; now on net CH115: D116.2 (A), J119.2, Q115.5 (D_1), Q115.6 (D_2), Q115.7 (D_3), Q115.8 (D_4), Q115.9 (D_5)
- net SOL116- is gone; now on net CH116: D117.2 (A), J120.2, Q116.5 (D_1), Q116.6 (D_2), Q116.7 (D_3), Q116.8 (D_4), Q116.9 (D_5)
- net SOL117- is gone; now on net CH117: D118.2 (A), J115.2, Q117.5 (D_1), Q117.6 (D_2), Q117.7 (D_3), Q117.8 (D_4), Q117.9 (D_5)
- net SOL118- is gone; now on net CH118: D119.2 (A), J121.2, Q118.5 (D_1), Q118.6 (D_2), Q118.7 (D_3), Q118.8 (D_4), Q118.9 (D_5)
- net SOL119- is gone; now on net CH119: D120.2 (A), J126.2, Q119.5 (D_1), Q119.6 (D_2), Q119.7 (D_3), Q119.8 (D_4), Q119.9 (D_5)
- net SOL120- is gone; now on net CH120: D121.2 (A), J124.2, Q120.5 (D_1), Q120.6 (D_2), Q120.7 (D_3), Q120.8 (D_4), Q120.9 (D_5)
- net SOL121- is gone; now on net CH121: D122.2 (A), J122.2, Q121.5 (D_1), Q121.6 (D_2), Q121.7 (D_3), Q121.8 (D_4), Q121.9 (D_5)
- net SOL122- is gone; now on net CH122: D123.2 (A), J127.2, Q122.5 (D_1), Q122.6 (D_2), Q122.7 (D_3), Q122.8 (D_4), Q122.9 (D_5)
- net SOL123- is gone; now on net CH123: D124.2 (A), J125.2, Q123.5 (D_1), Q123.6 (D_2), Q123.7 (D_3), Q123.8 (D_4), Q123.9 (D_5)
- net SOL124- is gone; now on net CH124: D125.2 (A), J123.2, Q124.5 (D_1), Q124.6 (D_2), Q124.7 (D_3), Q124.8 (D_4), Q124.9 (D_5)
- net SOL125- is gone; now on net CH125: D126.2 (A), J128.2, Q125.5 (D_1), Q125.6 (D_2), Q125.7 (D_3), Q125.8 (D_4), Q125.9 (D_5)
- net SOL126- is gone; now on net CH126: D127.2 (A), J129.2, Q126.5 (D_1), Q126.6 (D_2), Q126.7 (D_3), Q126.8 (D_4), Q126.9 (D_5)
- net SOL127- is gone; now on net CH127: D128.2 (A), J132.2, Q127.5 (D_1), Q127.6 (D_2), Q127.7 (D_3), Q127.8 (D_4), Q127.9 (D_5)
- net SOL128- is gone; now on net CH128: D129.2 (A), J133.2, Q128.5 (D_1), Q128.6 (D_2), Q128.7 (D_3), Q128.8 (D_4), Q128.9 (D_5)
- net SOL129- is gone; now on net CH129: D130.2 (A), J134.2, Q129.5 (D_1), Q129.6 (D_2), Q129.7 (D_3), Q129.8 (D_4), Q129.9 (D_5)
- net SOL130- is gone; now on net CH130: D131.2 (A), J130.2, Q130.5 (D_1), Q130.6 (D_2), Q130.7 (D_3), Q130.8 (D_4), Q130.9 (D_5)
- net SOL131- is gone; now on net CH131: D132.2 (A), J135.2, Q131.5 (D_1), Q131.6 (D_2), Q131.7 (D_3), Q131.8 (D_4), Q131.9 (D_5)
- net SOL132- is gone; now on net CH132: D133.2 (A), J136.2, Q132.5 (D_1), Q132.6 (D_2), Q132.7 (D_3), Q132.8 (D_4), Q132.9 (D_5)
- net SOL133- is gone; now on net CH133: D134.2 (A), J131.2, Q133.5 (D_1), Q133.6 (D_2), Q133.7 (D_3), Q133.8 (D_4), Q133.9 (D_5)
- net SOL134- is gone; now on net CH134: D135.2 (A), J137.2, Q134.5 (D_1), Q134.6 (D_2), Q134.7 (D_3), Q134.8 (D_4), Q134.9 (D_5)
- net SOL135- is gone; now on net CH135: D136.2 (A), J139.2, Q135.5 (D_1), Q135.6 (D_2), Q135.7 (D_3), Q135.8 (D_4), Q135.9 (D_5)
- net SOL136- is gone; now on net CH136: D137.2 (A), J140.2, Q136.5 (D_1), Q136.6 (D_2), Q136.7 (D_3), Q136.8 (D_4), Q136.9 (D_5)
- net SOL137- is gone; now on net CH137: D138.2 (A), J141.2, Q137.5 (D_1), Q137.6 (D_2), Q137.7 (D_3), Q137.8 (D_4), Q137.9 (D_5)
- net SOL138- is gone; now on net CH138: D139.2 (A), J138.2, Q138.5 (D_1), Q138.6 (D_2), Q138.7 (D_3), Q138.8 (D_4), Q138.9 (D_5)
- net SOL139- is gone; now on net CH139: D140.2 (A), J142.2, Q139.5 (D_1), Q139.6 (D_2), Q139.7 (D_3), Q139.8 (D_4), Q139.9 (D_5)
- net SOL140- is gone; now on net CH140: D141.2 (A), J143.2, Q140.5 (D_1), Q140.6 (D_2), Q140.7 (D_3), Q140.8 (D_4), Q140.9 (D_5)
- net SOL33- is gone; now on net CH33: D26.2 (A), J40.2, Q25.5 (D_1), Q25.6 (D_2), Q25.7 (D_3), Q25.8 (D_4), Q25.9 (D_5)
- net SOL34- is gone; now on net CH34: D27.2 (A), J41.2, Q26.5 (D_1), Q26.6 (D_2), Q26.7 (D_3), Q26.8 (D_4), Q26.9 (D_5)
- net SOL35- is gone; now on net CH35: D28.2 (A), J42.2, Q27.5 (D_1), Q27.6 (D_2), Q27.7 (D_3), Q27.8 (D_4), Q27.9 (D_5)
- net SOL36- is gone; now on net CH36: D29.2 (A), J43.2, Q28.5 (D_1), Q28.6 (D_2), Q28.7 (D_3), Q28.8 (D_4), Q28.9 (D_5)
- net SOL37- is gone; now on net CH37: D30.2 (A), J44.2, Q29.5 (D_1), Q29.6 (D_2), Q29.7 (D_3), Q29.8 (D_4), Q29.9 (D_5)
- net SOL38- is gone; now on net CH38: D31.2 (A), J45.2, Q30.5 (D_1), Q30.6 (D_2), Q30.7 (D_3), Q30.8 (D_4), Q30.9 (D_5)
- net SOL39- is gone; now on net CH39: D32.2 (A), J46.2, Q31.5 (D_1), Q31.6 (D_2), Q31.7 (D_3), Q31.8 (D_4), Q31.9 (D_5)
- net SOL40- is gone; now on net CH40: D33.2 (A), J47.2, Q32.5 (D_1), Q32.6 (D_2), Q32.7 (D_3), Q32.8 (D_4), Q32.9 (D_5)
- net SOL41- is gone; now on net CH41: D34.2 (A), J48.2, Q33.5 (D_1), Q33.6 (D_2), Q33.7 (D_3), Q33.8 (D_4), Q33.9 (D_5)
- net SOL42- is gone; now on net CH42: D35.2 (A), J49.2, Q34.5 (D_1), Q34.6 (D_2), Q34.7 (D_3), Q34.8 (D_4), Q34.9 (D_5)
- net SOL43- is gone; now on net CH43: D36.2 (A), J50.2, Q35.5 (D_1), Q35.6 (D_2), Q35.7 (D_3), Q35.8 (D_4), Q35.9 (D_5)
- net SOL44- is gone; now on net CH44: D37.2 (A), J51.2, Q36.5 (D_1), Q36.6 (D_2), Q36.7 (D_3), Q36.8 (D_4), Q36.9 (D_5)
- net SOL45- is gone; now on net CH45: D38.2 (A), J52.2, Q37.5 (D_1), Q37.6 (D_2), Q37.7 (D_3), Q37.8 (D_4), Q37.9 (D_5)
- net SOL46- is gone; now on net CH46: D39.2 (A), J53.2, Q38.5 (D_1), Q38.6 (D_2), Q38.7 (D_3), Q38.8 (D_4), Q38.9 (D_5)
- net SOL47- is gone; now on net CH47: D40.2 (A), J54.2, Q39.5 (D_1), Q39.6 (D_2), Q39.7 (D_3), Q39.8 (D_4), Q39.9 (D_5)
- net SOL48- is gone; now on net CH48: D41.2 (A), J55.2, Q40.5 (D_1), Q40.6 (D_2), Q40.7 (D_3), Q40.8 (D_4), Q40.9 (D_5)
- net SOL49- is gone; now on net CH49: D42.2 (A), J6.2, Q41.5 (D_1), Q41.6 (D_2), Q41.7 (D_3), Q41.8 (D_4), Q41.9 (D_5)
- net SOL50- is gone; now on net CH50: D43.2 (A), J4.2, Q42.5 (D_1), Q42.6 (D_2), Q42.7 (D_3), Q42.8 (D_4), Q42.9 (D_5)
- net SOL51- is gone; now on net CH51: D44.2 (A), J1.2, Q43.5 (D_1), Q43.6 (D_2), Q43.7 (D_3), Q43.8 (D_4), Q43.9 (D_5)
- net SOL52- is gone; now on net CH52: D45.2 (A), J7.2, Q44.5 (D_1), Q44.6 (D_2), Q44.7 (D_3), Q44.8 (D_4), Q44.9 (D_5)
- net SOL53- is gone; now on net CH53: D46.2 (A), J5.2, Q45.5 (D_1), Q45.6 (D_2), Q45.7 (D_3), Q45.8 (D_4), Q45.9 (D_5)
- net SOL54- is gone; now on net CH54: D47.2 (A), J2.2, Q46.5 (D_1), Q46.6 (D_2), Q46.7 (D_3), Q46.8 (D_4), Q46.9 (D_5)
- net SOL55- is gone; now on net CH55: D48.2 (A), J56.2, Q47.5 (D_1), Q47.6 (D_2), Q47.7 (D_3), Q47.8 (D_4), Q47.9 (D_5)
- net SOL56- is gone; now on net CH56: D49.2 (A), J57.2, Q48.5 (D_1), Q48.6 (D_2), Q48.7 (D_3), Q48.8 (D_4), Q48.9 (D_5)
- net SOL57- is gone; now on net CH57: D50.2 (A), J60.2, Q49.5 (D_1), Q49.6 (D_2), Q49.7 (D_3), Q49.8 (D_4), Q49.9 (D_5)
- net SOL58- is gone; now on net CH58: D51.2 (A), J61.2, Q50.5 (D_1), Q50.6 (D_2), Q50.7 (D_3), Q50.8 (D_4), Q50.9 (D_5)
- net SOL59- is gone; now on net CH59: D52.2 (A), J62.2, Q51.5 (D_1), Q51.6 (D_2), Q51.7 (D_3), Q51.8 (D_4), Q51.9 (D_5)
- net SOL60- is gone; now on net CH60: D53.2 (A), J58.2, Q52.5 (D_1), Q52.6 (D_2), Q52.7 (D_3), Q52.8 (D_4), Q52.9 (D_5)
- net SOL61- is gone; now on net CH61: D54.2 (A), J63.2, Q53.5 (D_1), Q53.6 (D_2), Q53.7 (D_3), Q53.8 (D_4), Q53.9 (D_5)
- net SOL62- is gone; now on net CH62: D55.2 (A), J64.2, Q54.5 (D_1), Q54.6 (D_2), Q54.7 (D_3), Q54.8 (D_4), Q54.9 (D_5)
- net SOL63- is gone; now on net CH63: D56.2 (A), J59.2, Q55.5 (D_1), Q55.6 (D_2), Q55.7 (D_3), Q55.8 (D_4), Q55.9 (D_5)
- net SOL64- is gone; now on net CH64: D57.2 (A), J65.2, Q56.5 (D_1), Q56.6 (D_2), Q56.7 (D_3), Q56.8 (D_4), Q56.9 (D_5)
- net SOL65- is gone; now on net CH65: D58.2 (A), J67.2, Q57.5 (D_1), Q57.6 (D_2), Q57.7 (D_3), Q57.8 (D_4), Q57.9 (D_5)
- net SOL66- is gone; now on net CH66: D59.2 (A), J68.2, Q58.5 (D_1), Q58.6 (D_2), Q58.7 (D_3), Q58.8 (D_4), Q58.9 (D_5)
- net SOL67- is gone; now on net CH67: D60.2 (A), J69.2, Q59.5 (D_1), Q59.6 (D_2), Q59.7 (D_3), Q59.8 (D_4), Q59.9 (D_5)
- net SOL68- is gone; now on net CH68: D61.2 (A), J66.2, Q60.5 (D_1), Q60.6 (D_2), Q60.7 (D_3), Q60.8 (D_4), Q60.9 (D_5)
- net SOL69- is gone; now on net CH69: D62.2 (A), J70.2, Q61.5 (D_1), Q61.6 (D_2), Q61.7 (D_3), Q61.8 (D_4), Q61.9 (D_5)
- net SOL70- is gone; now on net CH70: D63.2 (A), J71.2, Q62.5 (D_1), Q62.6 (D_2), Q62.7 (D_3), Q62.8 (D_4), Q62.9 (D_5)
- net SOL71- is gone; now on net CH71: D64.2 (A), J76.2, Q63.5 (D_1), Q63.6 (D_2), Q63.7 (D_3), Q63.8 (D_4), Q63.9 (D_5)
- net SOL72- is gone; now on net CH72: D65.2 (A), J77.2, Q64.5 (D_1), Q64.6 (D_2), Q64.7 (D_3), Q64.8 (D_4), Q64.9 (D_5)
- net SOL73- is gone; now on net CH73: D66.2 (A), J78.2, Q65.5 (D_1), Q65.6 (D_2), Q65.7 (D_3), Q65.8 (D_4), Q65.9 (D_5)
- net SOL74- is gone; now on net CH74: D67.2 (A), J79.2, Q66.5 (D_1), Q66.6 (D_2), Q66.7 (D_3), Q66.8 (D_4), Q66.9 (D_5)
- net SOL75- is gone; now on net CH75: D68.2 (A), J72.2, Q67.5 (D_1), Q67.6 (D_2), Q67.7 (D_3), Q67.8 (D_4), Q67.9 (D_5)
- net SOL76- is gone; now on net CH76: D69.2 (A), J73.2, Q68.5 (D_1), Q68.6 (D_2), Q68.7 (D_3), Q68.8 (D_4), Q68.9 (D_5)
- net SOL77- is gone; now on net CH77: D70.2 (A), J74.2, Q69.5 (D_1), Q69.6 (D_2), Q69.7 (D_3), Q69.8 (D_4), Q69.9 (D_5)
- net SOL78- is gone; now on net CH78: D71.2 (A), J75.2, Q70.5 (D_1), Q70.6 (D_2), Q70.7 (D_3), Q70.8 (D_4), Q70.9 (D_5)
- net SOL79- is gone; now on net CH79: D72.2 (A), J82.2, Q71.5 (D_1), Q71.6 (D_2), Q71.7 (D_3), Q71.8 (D_4), Q71.9 (D_5)
- net SOL82- is gone; now on net CH82: D75.2 (A), J85.2, Q74.5 (D_1), Q74.6 (D_2), Q74.7 (D_3), Q74.8 (D_4), Q74.9 (D_5)
- net SOL83- is gone; now on net CH83: D76.2 (A), J86.2, Q75.5 (D_1), Q75.6 (D_2), Q75.7 (D_3), Q75.8 (D_4), Q75.9 (D_5)
- net SOL84- is gone; now on net CH84: D77.2 (A), J81.2, Q76.5 (D_1), Q76.6 (D_2), Q76.7 (D_3), Q76.8 (D_4), Q76.9 (D_5)
- net SOL85- is gone; now on net CH85: D78.2 (A), J80.2, Q77.5 (D_1), Q77.6 (D_2), Q77.7 (D_3), Q77.8 (D_4), Q77.9 (D_5)
- net SOL86- is gone; now on net CH86: D79.2 (A), J87.2, Q78.5 (D_1), Q78.6 (D_2), Q78.7 (D_3), Q78.8 (D_4), Q78.9 (D_5)
- net SOL87- is gone; now on net CH87: D80.2 (A), J88.2, Q79.5 (D_1), Q79.6 (D_2), Q79.7 (D_3), Q79.8 (D_4), Q79.9 (D_5)
- net SOL88- is gone; now on net CH88: D81.2 (A), J89.2, Q80.5 (D_1), Q80.6 (D_2), Q80.7 (D_3), Q80.8 (D_4), Q80.9 (D_5)
- net SOL89- is gone; now on net CH89: D82.2 (A), J90.2, Q81.5 (D_1), Q81.6 (D_2), Q81.7 (D_3), Q81.8 (D_4), Q81.9 (D_5)
- net SOL90- is gone; now on net CH90: D83.2 (A), J91.2, Q82.5 (D_1), Q82.6 (D_2), Q82.7 (D_3), Q82.8 (D_4), Q82.9 (D_5)
- net SOL91- is gone; now on net CH91: D84.2 (A), J92.2, Q83.5 (D_1), Q83.6 (D_2), Q83.7 (D_3), Q83.8 (D_4), Q83.9 (D_5)
- net SOL92- is gone; now on net CH92: D85.2 (A), J93.2, Q84.5 (D_1), Q84.6 (D_2), Q84.7 (D_3), Q84.8 (D_4), Q84.9 (D_5)
- net SOL93- is gone; now on net CH93: D86.2 (A), J94.2, Q85.5 (D_1), Q85.6 (D_2), Q85.7 (D_3), Q85.8 (D_4), Q85.9 (D_5)
- net SOL94- is gone; now on net CH94: D87.2 (A), J95.2, Q86.5 (D_1), Q86.6 (D_2), Q86.7 (D_3), Q86.8 (D_4), Q86.9 (D_5)
- net SOL95- is gone; now on net CH95: D88.2 (A), J96.2, Q87.5 (D_1), Q87.6 (D_2), Q87.7 (D_3), Q87.8 (D_4), Q87.9 (D_5)
- net SOL96- is gone; now on net CH96: D89.2 (A), J97.2, Q88.5 (D_1), Q88.6 (D_2), Q88.7 (D_3), Q88.8 (D_4), Q88.9 (D_5)
- net SOL97- is gone; now on net CH97: D90.2 (A), J98.2, Q89.5 (D_1), Q89.6 (D_2), Q89.7 (D_3), Q89.8 (D_4), Q89.9 (D_5)
- net SOL98- is gone; now on net CH98: D91.2 (A), J99.2, Q90.5 (D_1), Q90.6 (D_2), Q90.7 (D_3), Q90.8 (D_4), Q90.9 (D_5)
- net SOL99- is gone; now on net CH99: D92.2 (A), J100.2, Q91.5 (D_1), Q91.6 (D_2), Q91.7 (D_3), Q91.8 (D_4), Q91.9 (D_5)
- net 5V_4: now also U69.1
- net 5V_5: no longer U69.1
- net SOL80- renamed 80
- net SOL81- renamed 81
