File: NozzleControlBoard.kicad_sch (KiCad schematic)
At the start: 1284 parts, among them IC2 MAX3094EESE+, IC3 MAX22245BAWA+, J1 SOL51, J10 SOL3, J100 SOL99, J101 SOL100, J102 SOL101, J103 SHIFT_DATA_TOSS, J104 8BIT_24V_OUT, J105 SOL102, J106 SOL105, J107 SOL108, J108 SOL104, J109 SOL107, J11 SOL4, J110 SOL103, J111 SOL106, J112 SOL109, J113 SOL110, J114 SOL114, J115 SOL117, J116 SOL111, J117 SOL112, J118 SOL113, J119 SOL115, J12 SOL5, J120 SOL116, J121 SOL118, J122 SOL121, J123 SOL124, J124 SOL120, J125 SOL123, J126 SOL119, J127 SOL122, J128 SOL125, J129 SOL126, J13 SOL6, J130 SOL130, J131 SOL133, J132 SOL127, J133 SOL128, J134 SOL129, J135 SOL131, J136 SOL132, J137 SOL134, J138 SOL138, J139 SOL135, J14 SOL7, J140 SOL136, J141 SOL137, J142 SOL139, J143 SOL140, J144 SHIFT_DATA_TOSS, J145 8BIT_24V_OUT, J15 SOL8, J16 SOL9, J17 SOL10, J18 SOL11, J19 SOL12, J2 SOL54, J20 SOL13, J21 SOL14, J22 SOL15, J23 SOL16, J24 SOL17, J25 SOL18, J26 SOL19, J27 SOL20, J28 SOL21, J29 SOL22, J3 Conn_01x12_Male, J30 SOL23, J31 SOL24, J32 SOL25, J33 SOL26, J34 SOL27, J35 SOL28, J36 SOL29, J37 SOL30, J38 SOL31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

Commit message: 이은혜
4/11
Connections:
- net 80 is gone; now on net CH80: D73.2 (A), J83.2, Q72.5 (D_1), Q72.6 (D_2), Q72.7 (D_3), Q72.8 (D_4), Q72.9 (D_5)
- net 81 is gone; now on net CH81: D74.2 (A), J84.2, Q73.5 (D_1), Q73.6 (D_2), Q73.7 (D_3), Q73.8 (D_4), Q73.9 (D_5)
Changed lines of the file:
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@@
     (effects (font (size 1.27 1.27)) (justify left bottom))
   )
-  (label "80" (at 962.2653 613.41 0) (fields_autoplaced)
+  (label "CH80" (at 962.2653 613.41 0) (fields_autoplaced)
     (effects (font (size 1.27 1.27)) (justify left bottom))
   )
@@
     (effects (font (size 1.27 1.27)) (justify right bottom))
   )
-  (label "81" (at 962.5999 636.27 0) (fields_autoplaced)
-    (effects (font (size 1.27 1.27)) (justify left bottom))
-  )
+  (label "CH81" (at 962.5999 636.27 0) (fields_autoplaced)
+    (effects (font (size 1.27 1.27)) (justify left bottom))
+  )

Commit message: .
.
Parts:
- J104, J145: footprint 24V_PAD:24V_PAD -> footprint:24V_PAD
- U4: footprint footprint:TPN22006NHLQ -> Connector_PinHeader_2.00mm:PinHeader_1x04_P2.00mm_Vertical
Connections:
- net 5V_4: no longer J103.5 (Pin_5), U69.1, U70.1
- net 5V_5: now also U69.1, U70.1
- net DATA13: now also J103.1 (Pin_1); no longer J144.1 (Pin_1), U86.14 (SER)
- net DATA15: no longer J103.1 (Pin_1)
- net GND_3: no longer J144.6 (Pin_6)
- net GND_4: no longer J103.6 (Pin_6)
- removed net S: U168.6 (QG), U168.7 (QH), U68.6 (QG), U68.7 (QH)
- new net DATA13_2: J144.1 (Pin_1), U86.14 (SER)
Changed lines of the file:
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@@
     (effects (font (size 1.27 1.27)) (justify left bottom))
   )
-  (label "S" (at 2688.0165 814.69 0) (fields_autoplaced)
-    (effects (font (size 1.27 1.27)) (justify left bottom))
-  )
   (label "24V2_GND" (at 779.145 752.475 0) (fields_autoplaced)
     (effects (font (size 1.27 1.27)) (justify left bottom))
@@
     (effects (font (size 1.27 1.27)) (justify left bottom))
   )
-  (label "S" (at 2688.0165 817.23 0) (fields_autoplaced)
-    (effects (font (size 1.27 1.27)) (justify left bottom))
-  )
   (label "5V_4" (at 852.805 671.195 0) (fields_autoplaced)
     (effects (font (size 1.27 1.27)) (justify left bottom))
@@
     (effects (font (size 1.27 1.27)) (justify left bottom))
   )
-  (label "5V_4" (at 687.705 579.755 0) (fields_autoplaced)
+  (label "5V_5" (at 687.705 579.755 0) (fields_autoplaced)
     (effects (font (size 1.27 1.27)) (justify left bottom))
   )
@@
     (effects (font (size 1.27 1.27)) (justify left bottom))
   )
-  (label "5V_4" (at 687.705 602.615 0) (fields_autoplaced)
+  (label "5V_5" (at 687.705 602.615 0) (fields_autoplaced)
     (effects (font (size 1.27 1.27)) (justify left bottom))
   )
@@
     (effects (font (size 1.27 1.27)) (justify left bottom))
   )
-  (label "S" (at 2691.1915 367.65 0) (fields_autoplaced)
-    (effects (font (size 1.27 1.27)) (justify left bottom))
-  )
   (label "MOSI" (at 609.6 261.62 0) (fields_autoplaced)
     (effects (font (size 1.27 1.27)) (justify left bottom))
@@
     (effects (font (size 1.27 1.27)) (justify left bottom))
   )
-  (label "DATA13" (at 709.8921 795.655 0) (fields_autoplaced)
+  (label "DATA13_2" (at 709.8921 795.655 0) (fields_autoplaced)
     (effects (font (size 1.27 1.27)) (justify left bottom))
   )
@@
     (effects (font (size 1.27 1.27)) (justify left bottom))
   )
-  (label "DATA15" (at 2939.8022 237.49 0) (fields_autoplaced)
+  (label "DATA13" (at 2939.8022 237.49 0) (fields_autoplaced)
     (effects (font (size 1.27 1.27)) (justify left bottom))
   )
@@
     (effects (font (size 1.27 1.27)) (justify left bottom))
   )
-  (label "DATA13" (at 454.2728 654.685 180) (fields_autoplaced)
+  (label "DATA13_2" (at 454.2728 654.685 180) (fields_autoplaced)
     (effects (font (size 1.27 1.27)) (justify right bottom))
   )
@@
     (effects (font (size 1.27 1.27)) (justify left bottom))
   )
-  (label "5V_4" (at 2944.495 247.65 0) (fields_autoplaced)
-    (effects (font (size 1.27 1.27)) (justify left bottom))
-  )
   (label "S41" (at 1875.5367 138.43 0) (fields_autoplaced)
     (effects (font (size 1.27 1.27)) (justify left bottom))
@@
     (effects (font (size 1.27 1.27)) (justify left bottom))
   )
-  (label "GND_4" (at 2944.495 250.19 0) (fields_autoplaced)
-    (effects (font (size 1.27 1.27)) (justify left bottom))
-  )
   (label "24V2" (at 721.36 221.615 0) (fields_autoplaced)
     (effects (font (size 1.27 1.27)) (justify left bottom))
@@
     (effects (font (size 1.27 1.27)) (justify left bottom))
   )
-  (label "S" (at 2691.1915 365.11 0) (fields_autoplaced)
-    (effects (font (size 1.27 1.27)) (justify left bottom))
-  )
   (label "S94" (at 1255.6965 812.165 0) (fields_autoplaced)
     (effects (font (size 1.27 1.27)) (justify left bottom))
@@
     (effects (font (size 1.27 1.27)) (justify left bottom))
   )
-  (label "GND_3" (at 449.58 667.385 180) (fields_autoplaced)
-    (effects (font (size 1.27 1.27)) (justify right bottom))
-  )
   (label "24V2_GND" (at 1409.065 728.98 0) (fields_autoplaced)
     (effects (font (size 1.27 1.27)) (justify left bottom))
@@
       (effects (font (size 1.27 1.27)))
     )
-    (property "Footprint" "footprint:TPN22006NHLQ" (at 518.16 325.12 0)
+    (property "Footprint" "Connector_PinHeader_2.00mm:PinHeader_1x04_P2.00mm_Vertical" (at 518.16 325.12 0)
       (effects (font (size 1.27 1.27)) hide)
     )
@@
       (effects (font (size 1.27 1.27)))
     )
-    (property "Footprint" "24V_PAD:24V_PAD" (at 2964.815 270.51 0)
+    (property "Footprint" "footprint:24V_PAD" (at 2964.815 270.51 0)
       (effects (font (size 1.27 1.27)) hide)
     )
@@
       (effects (font (size 1.27 1.27)))
     )
-    (property "Footprint" "24V_PAD:24V_PAD" (at 429.26 687.705 0)
+    (property "Footprint" "footprint:24V_PAD" (at 429.26 687.705 0)
       (effects (font (size 1.27 1.27)) hide)
     )

Commit message: 이은혜
4/13
Connections:
- net 5V_3: no longer J144.8 (Pin_8), PS2.3 (+VIN_1), PS2.4 (+VIN_2)
- net 5V_4: no longer C100.2, C101.2, C102.1, C54.2, C56.2, C59.1, C61.2, C68.2, C69.1, C70.2, C71.2, C72.1, C73.2, C74.2, C75.1, C76.2, C77.2, C78.1, C79.2, C80.2, C81.1, C82.2, C83.2, C84.1, C85.2, C86.2, C87.1, C88.2, C89.2, C90.1, C91.2, C92.2, C93.1, C94.2, C95.2, C96.1, C97.2, C98.2, C99.1, U100.1, U101.1, U111.1, U112.1, U113.1, U114.10 (~{SRCLR}), U114.16 (VCC), U115.1, U116.1, U117.1, U118.1, U119.1, U120.1, U121.1, U122.1, U123.10 (~{SRCLR}), U123.16 (VCC), U124.20 (VCC), U125.1, U126.1, U127.1, U128.1, U129.1, U130.1, U131.1, U132.1, U133.10 (~{SRCLR}), U133.16 (VCC), U134.1, U135.1, U136.1, U137.1, U138.1, U139.1, U140.1, U141.1, U142.10 (~{SRCLR}), U142.16 (VCC), U143.20 (VCC), U144.1, U145.1, U146.1, U147.1, U148.1, U149.1, U150.1, U151.1, U152.10 (~{SRCLR}), U152.16 (VCC), U153.1, U154.1, U155.1, U156.1, U157.1, U158.1, U159.1, U160.1, U161.10 (~{SRCLR}), U161.16 (VCC), U162.1, U163.1, U164.1, U165.1, U166.1, U167.1, U168.10 (~{SRCLR}), U168.16 (VCC), U169.20 (VCC), U71.1, U72.1, U82.1, U83.1, U84.1, U85.1, U86.10 (~{SRCLR}), U86.16 (VCC), U87.1, U88.1, U89.1, U90.1, U91.1, U92.1, U93.1, U94.1, U95.10 (~{SRCLR}), U95.16 (VCC), U96.20 (VCC), U97.1, U98.1, U99.1
- net 5V_5: now also C100.2, C101.2, C102.1, C54.2, C56.2, C59.1, C61.2, C68.2, C69.1, C70.2, C71.2, C72.1, C73.2, C74.2, C75.1, C76.2, C77.2, C78.1, C79.2, C80.2, C81.1, C82.2, C83.2, C84.1, C85.2, C86.2, C87.1, C88.2, C89.2, C90.1, C91.2, C92.2, C93.1, C94.2, C95.2, C96.1, C97.2, C98.2, C99.1, U100.1, U101.1, U111.1, U112.1, U113.1, U114.10 (~{SRCLR}), U114.16 (VCC), U115.1, U116.1, U117.1, U118.1, U119.1, U120.1, U121.1, U122.1, U123.10 (~{SRCLR}), U123.16 (VCC), U124.20 (VCC), U125.1, U126.1, U127.1, U128.1, U129.1, U130.1, U131.1, U132.1, U133.10 (~{SRCLR}), U133.16 (VCC), U134.1, U135.1, U136.1, U137.1, U138.1, U139.1, U140.1, U141.1, U142.10 (~{SRCLR}), U142.16 (VCC), U143.20 (VCC), U144.1, U145.1, U146.1, U147.1, U148.1, U149.1, U150.1, U151.1, U152.10 (~{SRCLR}), U152.16 (VCC), U153.1, U154.1, U155.1, U156.1, U157.1, U158.1, U159.1, U160.1, U161.10 (~{SRCLR}), U161.16 (VCC), U162.1, U163.1, U164.1, U165.1, U166.1, U167.1, U168.10 (~{SRCLR}), U168.16 (VCC), U169.20 (VCC), U71.1, U72.1, U82.1, U83.1, U84.1, U85.1, U86.10 (~{SRCLR}), U86.16 (VCC), U87.1, U88.1, U89.1, U90.1, U91.1, U92.1, U93.1, U94.1, U95.10 (~{SRCLR}), U95.16 (VCC), U96.20 (VCC), U97.1, U98.1, U99.1
- net GND_3: no longer J144.7 (Pin_7), PS2.1 (-VIN_1), PS2.2 (-VIN_2), PS2.5 (SGNDIN_1), PS2.6 (SGNDIN_2), PS2.7 (SGNDIN_3), PS2.8 (SGNDIN_4)
- net GND_4: no longer C100.1, C101.1, C102.2, C54.1, C56.1, C59.2, C61.1, C68.1, C69.2, C70.1, C71.1, C72.2, C73.1, C74.1, C75.2, C76.1, C77.1, C78.2, C79.1, C80.1, C81.2, C82.1, C83.1, C84.2, C85.1, C86.1, C87.2, C88.1, C89.1, C90.2, C91.1, C92.1, C93.2, C94.1, C95.1, C96.2, C97.1, C98.1, C99.2, R270.1, R319.1, R368.1, R435.1, U114.8 (GND), U123.8 (GND), U124.10 (GND), U133.8 (GND), U142.8 (GND), U143.10 (GND), U152.8 (GND), U161.8 (GND), U168.8 (GND), U169.10 (GND), U86.8 (GND), U95.8 (GND), U96.10 (GND)
- net GND_5: now also C100.1, C101.1, C102.2, C54.1, C56.1, C59.2, C61.1, C68.1, C69.2, C70.1, C71.1, C72.2, C73.1, C74.1, C75.2, C76.1, C77.1, C78.2, C79.1, C80.1, C81.2, C82.1, C83.1, C84.2, C85.1, C86.1, C87.2, C88.1, C89.1, C90.2, C91.1, C92.1, C93.2, C94.1, C95.1, C96.2, C97.1, C98.1, C99.2, R270.1, R319.1, R368.1, R435.1, U114.8 (GND), U123.8 (GND), U124.10 (GND), U133.8 (GND), U142.8 (GND), U143.10 (GND), U152.8 (GND), U161.8 (GND), U168.8 (GND), U169.10 (GND), U86.8 (GND), U95.8 (GND), U96.10 (GND)
- new net 5V_6: J144.8 (Pin_8), PS2.3 (+VIN_1), PS2.4 (+VIN_2)
- new net GND_6: J144.7 (Pin_7), PS2.1 (-VIN_1), PS2.2 (-VIN_2), PS2.5 (SGNDIN_1), PS2.6 (SGNDIN_2), PS2.7 (SGNDIN_3), PS2.8 (SGNDIN_4)

Commit message: 이은혜
Connections:
- net 5V_4: no longer C47.2, C50.2, C52.1, U53.1, U54.1, U55.1, U65.1, U66.1, U67.1, U68.10 (~{SRCLR}), U68.16 (VCC)
- net 5V_5: now also C47.2, C50.2, C52.1, U53.1, U54.1, U55.1, U65.1, U66.1, U67.1, U68.10 (~{SRCLR}), U68.16 (VCC)
- net CLK_4: no longer U68.11 (SRCLK)
- net CLK_6: now also U68.11 (SRCLK)
- net DATA11: now also U52.8 (1A3); no longer U68.14 (SER)
- net DATA12: now also J103.1 (Pin_1), U52.12 (1Y3); no longer U52.8 (1A3), U68.9 (QH')
- net DATA13: now also J144.1 (Pin_1), U68.14 (SER); no longer J103.1 (Pin_1), U52.12 (1Y3)
- net DATA14: now also U68.9 (QH'), U86.14 (SER); no longer U86.9 (QH'), U95.14 (SER)
- net DATA15: now also U86.9 (QH'), U95.14 (SER); no longer U95.9 (QH'), U96.8 (1A3)
- net DATA16: now also U95.9 (QH'), U96.8 (1A3); no longer U114.14 (SER), U96.12 (1Y3)
- net DATA17: now also U114.14 (SER), U96.12 (1Y3); no longer U114.9 (QH'), U123.14 (SER)
- net DATA18: now also U114.9 (QH'), U123.14 (SER); no longer U123.9 (QH'), U124.8 (1A3)
- net DATA19: now also U123.9 (QH'), U124.8 (1A3); no longer U124.12 (1Y3), U133.14 (SER)
- net DATA20: now also U124.12 (1Y3), U133.14 (SER); no longer U133.9 (QH'), U142.14 (SER)
- net DATA21: now also U133.9 (QH'), U142.14 (SER); no longer U142.9 (QH'), U143.8 (1A3)
- net DATA22: now also U142.9 (QH'), U143.8 (1A3); no longer U143.12 (1Y3), U152.14 (SER)
- net DATA23: now also U143.12 (1Y3), U152.14 (SER); no longer U152.9 (QH')
- net DATA24: now also U152.9 (QH'); no longer U161.9 (QH'), U168.14 (SER)
- net DATA25: now also U161.9 (QH'), U168.14 (SER); no longer U168.9 (QH'), U169.8 (1A3)
- net DATA26: now also U168.9 (QH'), U169.8 (1A3); no longer U169.12 (1Y3)
- net ENABLE_4: no longer U68.13 (~{OE})
- net ENABLE_6: now also U68.13 (~{OE})
- net GND_4: no longer C47.1, C50.1, C52.2, U68.8 (GND)
- net GND_5: now also C47.1, C50.1, C52.2, U68.8 (GND)
- net LATCH_4: no longer U68.12 (RCLK)
- net LATCH_6: now also U68.12 (RCLK)
- removed net DATA13_2: J144.1 (Pin_1), U86.14 (SER)
- new net DATA27: U169.12 (1Y3)
